File: sd_hardware/sd_hardware.kicad_sch (KiCad schematic)
At the start: 12 parts, among them IC1 BD9E201FP4-Z, U1 STM32G431K8Tx

Commit message: add .
Parts:
- removed U1: STM32G431K8Tx, Package_QFP:LQFP-32_7x7mm_P0.8mm, symbol MCU_ST_STM32G4:STM32G431K8Tx
- added C1, C2: 1μ, symbol Device:C
- added D1, D19: LED, symbol Device:LED
- added J10, J3, J4, J5, J6, J7, J8, J9: Conn_01x02_Socket, symbol Connector:Conn_01x02_Socket
- added J11, J2: RJ45, symbol Connector:RJ45
- added PS1: BU33SD5WG-TR, SOT95P280X125-5N, symbol BU33SD5WG-TR:BU33SD5WG-TR
- added R1, R12: 1k, symbol Device:R
- renumbered C1 to C3, C2 to C4, C3 to C5, C4 to C6, C5 to C7, C6 to C8, D1 to D2, R1 to R2, R2 to R3
Connections:
- net +24V: now reaches C7.1, C8.1, IC1.3 (VIN)
- new net: D19.2 (A), R12.2
- new net: D1.2 (A), R1.2
- new net +3.3V: C2.1, PS1.5 (VOUT), R1.1, R12.1
- new net +5V: C1.1, J11.4, J11.5, J2.4, J2.5, PS1.1 (VIN), PS1.3 (STBY)
- new net CANH: J11.2, J11.6, J2.2, J2.6
- new net CANL: J11.1, J11.3, J2.1, J2.3
- new net GND: C1.2, C2.2, J11.7, J11.8, J2.7, J2.8, PS1.2 (GND)
- new net MCU_stm32_g431k8t6/FDCAN1_LED: D19.1 (K)
- new net MCU_stm32_g431k8t6/MCU_State_LED: D1.1 (K)
- new net Solenoid_Isolation/Solenoid1_+: J3.2 (Pin_2)
- new net Solenoid_Isolation/Solenoid1_-: J3.1 (Pin_1)
- new net Solenoid_Isolation/Solenoid2_+: J4.2 (Pin_2)
- new net Solenoid_Isolation/Solenoid2_-: J4.1 (Pin_1)
- new net Solenoid_Isolation/Solenoid3_+: J5.2 (Pin_2)
- new net Solenoid_Isolation/Solenoid3_-: J5.1 (Pin_1)
- new net Solenoid_Isolation/Solenoid4_+: J6.2 (Pin_2)
- new net Solenoid_Isolation/Solenoid4_-: J6.1 (Pin_1)
- new net Solenoid_Isolation/Solenoid5_+: J7.2 (Pin_2)
- new net Solenoid_Isolation/Solenoid5_-: J7.1 (Pin_1)
- new net Solenoid_Isolation/Solenoid6_+: J8.2 (Pin_2)
- new net Solenoid_Isolation/Solenoid6_-: J8.1 (Pin_1)
- new net Solenoid_Isolation/Solenoid7_+: J9.2 (Pin_2)
- new net Solenoid_Isolation/Solenoid7_-: J9.1 (Pin_1)
- new net Solenoid_Isolation/Solenoid8_+: J10.2 (Pin_2)
- new net Solenoid_Isolation/Solenoid8_-: J10.1 (Pin_1)
Other:
- sheet Iso_Solenoid1 renamed Solenoid_Isolation
- removed sheet Iso_Solenoid2
- removed sheet Iso_Solenoid3
- removed sheet Iso_Solenoid4
- removed sheet Iso_Solenoid5
- removed sheet Iso_Solenoid6
- removed sheet Iso_Solenoid7
- removed sheet Iso_Solenoid8
- added sheet FDCAN_Transceiver (FDCAN_Transceiver.kicad_sch)
- added sheet MCU_stm32_g431k8t6 (MCU_stm32_g431k8t6.kicad_sch)
- sheet Solenoid_Isolation: file ISO_Solenoid.kicad_sch -> Solenoid_Isolation.kicad_sch
- sheet Solenoid_Isolation ports: added GPIO1_IN, GPIO2_IN, GPIO3_IN, GPIO4_IN, GPIO5_IN, GPIO6_IN, GPIO7_IN, GPIO8_IN, Solenoid1_+, Solenoid1_-, Solenoid2_+, Solenoid2_-, Solenoid3_+, Solenoid3_-, Solenoid4_+, Solenoid4_-, Solenoid5_+, Solenoid5_-, Solenoid6_+, Solenoid6_-, Solenoid7_+, Solenoid7_-, Solenoid8_+, Solenoid8_-; removed GPIO_IN, Solenoid_+, Solenoid_-
- moved on the sheet: C3, C4, C5, C6, C7, C8, D2, IC1, L1, R2, R3
