File: sd_hardware/sd_hardware.kicad_sch (KiCad schematic)
At the start: 33 parts, among them IC1 BD9E201FP4-Z, J1 Conn_01x02_Socket, J10 RJ45, J11 XT60PW-M_1x02_Horizontal, J12 Conn_01x02_Socket, J15 Conn_01x06_Socket, J2 Conn_01x02_Socket, J3 Conn_01x02_Socket, J4 Conn_01x02_Socket, J5 Conn_01x02_Socket, J6 Conn_01x02_Socket, J7 Conn_01x02_Socket, J8 Conn_01x02_Socket, J9 RJ45, SW2 SW_DIP_x03

Commit message: created schematic
Parts:
- added R42, R43, R44: 0, Resistor_SMD:R_0603_1608Metric_Pad0.98x0.95mm_HandSolder, symbol Device:R
- J10: renamed from J15; footprint (none) -> Connector_JST:JST_XH_B6B-XH-A_1x06_P2.50mm_Vertical
- R5: renamed from R6; footprint (none) -> Resistor_SMD:R_0603_1608Metric_Pad0.98x0.95mm_HandSolder
- R6: renamed from R7; footprint (none) -> Resistor_SMD:R_0603_1608Metric_Pad0.98x0.95mm_HandSolder
- renumbered C9 to C1, C10 to C2, C11 to C3, C12 to C4, C13 to C5, C7 to C6, C8 to C7, D18 to D1, D19 to D2, D17 to D3, J12 to J11, J10 to J12, J9 to J13, J11 to J8, J8 to J9, R11 to R1, R12 to R2, R9 to R3, R10 to R4, SW2 to SW1
Connections:
- net SPI_ADC/VIN: now reaches J10.6 (Pin_6)
- new net MCU_stm32_g431k8t6/EP_Regu_ADC_CS: R43.1
- new net MCU_stm32_g431k8t6/EP_Regu_DAC_CS: R42.1
- new net SPI_ADC/MISO: R44.2
- new net SPI_Iso/CS1_IN: R42.2
- new net SPI_Iso/CS2_IN: R43.2
- new net SPI_Iso/MISO_IN: R44.1
Other:
- sheet MCU_stm32_g431k8t6 ports: added EP_Regu_ADC_CS, EP_Regu_DAC_CS; removed EP_Regu_LATCH
- sheet SPI_ADC ports: added CS_N, MISO, MOSI, SCLK, VIN; removed none
- sheet SPI_DAC ports: added CS_N; removed LATCH, SDO
- sheet SPI_Iso ports: added CS1_IN, CS1_OUT, CS2_IN, CS2_OUT; removed CS_IN, CS_OUT
- moved on the sheet: R5, R6

Commit message: working
Parts:
- added C13, C14: 1μ, Capacitor_SMD:C_0603_1608Metric_Pad1.08x0.95mm_HandSolder, symbol Device:C_Small
- added D20, D21: LED, LED_SMD:LED_0603_1608Metric_Pad1.05x0.95mm_HandSolder, symbol Device:LED
- added R33: 56.7k, Resistor_SMD:R_0603_1608Metric_Pad0.98x0.95mm_HandSolder, symbol Device:R
- added R34: 10k, Resistor_SMD:R_0603_1608Metric_Pad0.98x0.95mm_HandSolder, symbol Device:R
- added R50, R51: 1k, Resistor_SMD:R_0603_1608Metric_Pad0.98x0.95mm_HandSolder, symbol Device:R
- added U7: BD00FC0WEFJ, Package_SO:HTSOP-8-1EP_3.9x4.9mm_P1.27mm_EP2.4x3.2mm, symbol Regulator_Linear:BD00FC0WEFJ
- J12: renamed from J11; footprint Connector_JST:JST_XH_B2B-XH-AM_1x02_P2.50mm_Vertical -> Connector_JST:JST_XH_B2B-XH-A_1x02_P2.50mm_Vertical
- J2, J3, J4, J5, J6, J7: footprint Connector_JST:JST_XH_B2B-XH-AM_1x02_P2.50mm_Vertical -> Connector_JST:JST_XH_B2B-XH-A_1x02_P2.50mm_Vertical
- J8: renamed from J9; footprint Connector_JST:JST_XH_B2B-XH-AM_1x02_P2.50mm_Vertical -> Connector_JST:JST_XH_B2B-XH-A_1x02_P2.50mm_Vertical
- renumbered C5 to C10, C2 to C11, C3 to C12, C1 to C15, C6 to C7, C7 to C8, C4 to C9, D1 to D17, D2 to D18, D3 to D19, IC1 to IC9, J12 to J10, J13 to J11, J8 to J13, J10 to J14, R1 to R26, R2 to R27, R42 to R28, R43 to R29, R5 to R30, R6 to R31, R44 to R32, R3 to R35, R4 to R36, SW1 to SW2
Connections:
- net +24V: now also C13.1, U7.5 (EN), U7.8 (VCC)
- net +3.3V: now also R50.1
- net GND: now also D20.1 (K)
- net GNDPWR: now also C13.2, C14.2, D21.1 (K), R34.2, U7.3 (GND), U7.9 (GND)
- new net: D20.2 (A), R50.2
- new net: D21.2 (A), R51.2
- new net: R33.1, R34.1, U7.2 (FB)
- new net +5VP: C14.1, R33.2, R51.1, U7.1 (VO)
Other:
- moved on the sheet: C7, C8, J1, J10, J11, J13, J14, J2, J3, J4, J5, J6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

Commit message: working
Parts:
- added J15: Conn_01x04_Socket, Connector_JST:JST_XH_B4B-XH-A_1x04_P2.50mm_Vertical, symbol Connector:Conn_01x04_Socket
- added R52, R53, R54: 0, Resistor_SMD:R_0603_1608Metric_Pad0.98x0.95mm_HandSolder, symbol Device:R
- C11, C12: footprint Capacitor_SMD:C_0603_1608Metric_Pad1.08x0.95mm_HandSolder -> Capacitor_SMD:C_1210_3225Metric_Pad1.33x2.70mm_HandSolder
Connections:
- net +12V: now also J15.1 (Pin_1)
- net GNDPWR: now also J15.2 (Pin_2)
- net MCU_stm32_g431k8t6/SPI1_MISO: now also R52.1
- net SPI_ADC/MOSI: now also R53.2
- net SPI_ADC/SCLK: now also R54.2
- net SPI_ADC/VIN: now also J15.4 (Pin_4)
- net SPI_DAC/VOUT: now also J15.3 (Pin_3)
- new net SPI_Iso/CLK_OUT: R54.1
- new net SPI_Iso/MISO_OUT: R52.2
- new net SPI_Iso/MOSI_OUT: R53.1
Other:
- note added: "1. Brown Vs(+12V) 2. Blue GND 4. White Vin(DAC OUT) 6. Black Monitor"
- title: (none) -> Solenoid_Driver_3.1 - Yamana
- moved on the sheet: C13, C14, D21, R30, R31, R32, R33, R34, R51, U7
