File: sd_hardware/SPI_ADC.kicad_sch (KiCad schematic)
At the start: 9 parts, among them U1 ADS1018IDGSR

Commit message: created schematic
Parts:
- removed C18: 10μ, symbol Device:C
- removed C19, C20: 0.1μ, symbol Device:C
- removed R1, R38, R39: 4.7k, symbol Device:R
- added C22: 0.1μ, Capacitor_SMD:C_0603_1608Metric_Pad1.08x0.95mm_HandSolder, symbol Device:C
- added C23: 10nF, Capacitor_SMD:C_0603_1608Metric_Pad1.08x0.95mm_HandSolder, symbol Device:C
- added R45, R47: 100k, Resistor_SMD:R_0603_1608Metric_Pad0.98x0.95mm_HandSolder, symbol Device:R
- added U5: BD87581YG-C, y-robo_footprint:SOT95P280X125-5N, symbol y-robo:BD87581YG-C
- C21: renamed from C17; footprint (none) -> Capacitor_SMD:C_0603_1608Metric_Pad1.08x0.95mm_HandSolder
- R46: renamed from R40; footprint (none) -> Resistor_SMD:R_0603_1608Metric_Pad0.98x0.95mm_HandSolder
- U6: renamed from U1; footprint DGS0010A_N -> y-robo_footprint:DGS10_TEX
Connections:
- net +5VP: now also U5.5 (V+)
- net GNDPWR: now also C22.2, C23.2, R47.2, U5.2 (V-)
- net VIN: now also R45.1
- net at R46.1: now also U5.3 (-), U5.4
- net at R46.2, U6.4 (AIN0): now also C23.1
- new net: C22.1, R45.2, R47.1, U5.1 (+)
Other:
- note added: "Vin (1~5V)↓ OP V+ (0.5~2.5V)"
- note removed: "Vin (1~5V)↓ Ain0 (0.5~2.5V)"
- moved on the sheet: C21, R46

Commit message: working
Parts:
- renumbered C21 to C23, C22 to C24, C23 to C25, R45 to R47, R46 to R48, R47 to R49
Changed lines of the file:
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@@
 		(dnp no)
 		(fields_autoplaced yes)
-		(property "Reference" "R45"
+		(property "Reference" "R47"
 			(at 53.34 74.9299 0)
 			(show_name no)
@@
 			(project "sd_hardware"
 				(path "/f972cb7f-90df-45d5-98d4-dc82335c3d91/a2cbaed3-dfb5-44af-a359-033db6a4bd15"
-					(reference "R45")
+					(reference "R47")
 					(unit 1)
 				)
@@
 		(dnp no)
 		(fields_autoplaced yes)
-		(property "Reference" "#PWR055"
+		(property "Reference" "#PWR0158"
 			(at 111.76 102.87 0)
 			(hide yes)
@@
 			(project "sd_hardware"
 				(path "/f972cb7f-90df-45d5-98d4-dc82335c3d91/a2cbaed3-dfb5-44af-a359-033db6a4bd15"
-					(reference "#PWR055")
+					(reference "#PWR0158")
 					(unit 1)
 				)
@@
 		(dnp no)
 		(fields_autoplaced yes)
-		(property "Reference" "#PWR053"
+		(property "Reference" "#PWR0156"
 			(at 77.47 74.93 0)
 			(hide yes)
@@
 			(project "sd_hardware"
 				(path "/f972cb7f-90df-45d5-98d4-dc82335c3d91/a2cbaed3-dfb5-44af-a359-033db6a4bd15"
-					(reference "#PWR053")
+					(reference "#PWR0156")
 					(unit 1)
 				)
@@
 		(dnp no)
 		(fields_autoplaced yes)
-		(property "Reference" "#PWR054"
+		(property "Reference" "#PWR0157"
 			(at 175.26 101.6 0)
 			(hide yes)
@@
 			(project "sd_hardware"
 				(path "/f972cb7f-90df-45d5-98d4-dc82335c3d91/a2cbaed3-dfb5-44af-a359-033db6a4bd15"
-					(reference "#PWR054")
+					(reference "#PWR0157")
 					(unit 1)
 				)
@@
 		(dnp no)
 		(fields_autoplaced yes)
-		(property "Reference" "R47"
+		(property "Reference" "R49"
 			(at 53.34 85.0899 0)
 			(show_name no)
@@
 			(project "sd_hardware"
 				(path "/f972cb7f-90df-45d5-98d4-dc82335c3d91/a2cbaed3-dfb5-44af-a359-033db6a4bd15"
-					(reference "R47")
+					(reference "R49")
 					(unit 1)
 				)
@@
 		(in_pos_files yes)
 		(dnp no)
-		(property "Reference" "C22"
+		(property "Reference" "C24"
 			(at 64.008 85.09 0)
 			(show_name no)
@@
 			(project "sd_hardware"
 				(path "/f972cb7f-90df-45d5-98d4-dc82335c3d91/a2cbaed3-dfb5-44af-a359-033db6a4bd15"
-					(reference "C22")
+					(reference "C24")
 					(unit 1)
 				)
@@
 		(dnp no)
 		(fields_autoplaced yes)
-		(property "Reference" "C23"
+		(property "Reference" "C25"
 			(at 107.95 87.6299 0)
 			(show_name no)
@@
 			(project "sd_hardware"
 				(path "/f972cb7f-90df-45d5-98d4-dc82335c3d91/a2cbaed3-dfb5-44af-a359-033db6a4bd15"
-					(reference "C23")
+					(reference "C25")
 					(unit 1)
 				)
@@
 		(dnp no)
 		(fields_autoplaced yes)
-		(property "Reference" "C21"
+		(property "Reference" "C23"
 			(at 123.19 55.8799 0)
 			(show_name no)
@@
 			(project "sd_hardware"
 				(path "/f972cb7f-90df-45d5-98d4-dc82335c3d91/a2cbaed3-dfb5-44af-a359-033db6a4bd15"
-					(reference "C21")
+					(reference "C23")
 					(unit 1)
 				)
@@
 		(dnp no)
 		(fields_autoplaced yes)
-		(property "Reference" "#PWR052"
+		(property "Reference" "#PWR0155"
 			(at 113.03 68.58 0)
 			(hide yes)
@@
 			(project "sd_hardware"
 				(path "/f972cb7f-90df-45d5-98d4-dc82335c3d91/a2cbaed3-dfb5-44af-a359-033db6a4bd15"
-					(reference "#PWR052")
+					(reference "#PWR0155")
 					(unit 1)
 				)
@@
 		(in_pos_files yes)
 		(dnp no)
-		(property "Reference" "R46"
+		(property "Reference" "R48"
 			(at 91.694 82.55 90)
 			(show_name no)
@@
 			(project "sd_hardware"
 				(path "/f972cb7f-90df-45d5-98d4-dc82335c3d91/a2cbaed3-dfb5-44af-a359-033db6a4bd15"
-					(reference "R46")
+					(reference "R48")
 					(unit 1)
 				)
@@
 		(dnp no)
 		(fields_autoplaced yes)
-		(property "Reference" "#PWR051"
+		(property "Reference" "#PWR0154"
 			(at 113.03 54.61 0)
 			(hide yes)
@@
 			(project "sd_hardware"
 				(path "/f972cb7f-90df-45d5-98d4-dc82335c3d91/a2cbaed3-dfb5-44af-a359-033db6a4bd15"
-					(reference "#PWR051")
-					(unit 1)
-				)
+					(reference "#PWR0154")
+					(unit 1)
+				)

Commit message: working
Other:
- title: (none) -> Solenoid_Driver_3.1 - Yamana
Changed lines of the file:
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@@
 	(generator_version "10.0")
 	(paper "A4")
+	(title_block
+		(title "Solenoid_Driver_3.1 - Yamana")
+		(date "2026-10-18")
+	)
 	(text "Vin (1~5V)↓\nOP V+ (0.5~2.5V)"
 		(exclude_from_sim no)
