File: sd_hardware/SPI_Iso.kicad_sch (KiCad schematic)
At the start: 8 parts, among them U2 ADUM251N1BRIZ

Commit message: created schematic
Parts:
- removed R4, R5, R8: 0, symbol Device:R
- C19: renamed from C21; footprint RW-16_ADI -> Capacitor_SMD:C_0603_1608Metric_Pad1.08x0.95mm_HandSolder
- C20: renamed from C22; footprint RW-16_ADI -> Capacitor_SMD:C_0603_1608Metric_Pad1.08x0.95mm_HandSolder
- R40: renamed from R2; footprint (none) -> Resistor_SMD:R_0603_1608Metric_Pad0.98x0.95mm_HandSolder
- R41: renamed from R3; footprint (none) -> Resistor_SMD:R_0603_1608Metric_Pad0.98x0.95mm_HandSolder
- U4: renamed from U2; footprint ADUM251N1BRIZ_ADI -> y-robo_footprint:ADUM251N1BRIZ_ADI
Connections:
- net CS1_IN: now also R40.2, U4.2 (VIA)
- net CS2_IN: now also R41.2, U4.3 (VIB)
- net MISO_IN: now also U4.11 (VIE)

Commit message: working
Parts:
- renumbered C19 to C18, C20 to C19, R40 to R37, R41 to R38, U4 to U2
Changed lines of the file:
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@@
 		(dnp no)
 		(fields_autoplaced yes)
-		(property "Reference" "#PWR048"
+		(property "Reference" "#PWR0151"
 			(at 171.45 74.93 0)
 			(hide yes)
@@
 			(project "sd_hardware"
 				(path "/f972cb7f-90df-45d5-98d4-dc82335c3d91/898550ec-f46f-4748-8c3b-5dbafb3c9cde"
-					(reference "#PWR048")
+					(reference "#PWR0151")
 					(unit 1)
 				)
@@
 		(dnp no)
 		(fields_autoplaced yes)
-		(property "Reference" "R41"
+		(property "Reference" "R38"
 			(at 104.14 77.4699 0)
 			(show_name no)
@@
 			(project "sd_hardware"
 				(path "/f972cb7f-90df-45d5-98d4-dc82335c3d91/898550ec-f46f-4748-8c3b-5dbafb3c9cde"
-					(reference "R41")
+					(reference "R38")
 					(unit 1)
 				)
@@
 		(dnp no)
 		(fields_autoplaced yes)
-		(property "Reference" "#PWR049"
+		(property "Reference" "#PWR0152"
 			(at 110.49 114.3 0)
 			(hide yes)
@@
 			(project "sd_hardware"
 				(path "/f972cb7f-90df-45d5-98d4-dc82335c3d91/898550ec-f46f-4748-8c3b-5dbafb3c9cde"
-					(reference "#PWR049")
+					(reference "#PWR0152")
 					(unit 1)
 				)
@@
 		(dnp no)
 		(fields_autoplaced yes)
-		(property "Reference" "C20"
+		(property "Reference" "C19"
 			(at 167.64 77.4699 0)
 			(show_name no)
@@
 			(project "sd_hardware"
 				(path "/f972cb7f-90df-45d5-98d4-dc82335c3d91/898550ec-f46f-4748-8c3b-5dbafb3c9cde"
-					(reference "C20")
+					(reference "C19")
 					(unit 1)
 				)
@@
 		(dnp no)
 		(fields_autoplaced yes)
-		(property "Reference" "U4"
+		(property "Reference" "U2"
 			(at 139.7 72.39 0)
 			(show_name no)
@@
 			(project "sd_hardware"
 				(path "/f972cb7f-90df-45d5-98d4-dc82335c3d91/898550ec-f46f-4748-8c3b-5dbafb3c9cde"
-					(reference "U4")
+					(reference "U2")
 					(unit 1)
 				)
@@
 		(dnp no)
 		(fields_autoplaced yes)
-		(property "Reference" "#PWR047"
+		(property "Reference" "#PWR0150"
 			(at 92.71 73.66 0)
 			(hide yes)
@@
 			(project "sd_hardware"
 				(path "/f972cb7f-90df-45d5-98d4-dc82335c3d91/898550ec-f46f-4748-8c3b-5dbafb3c9cde"
-					(reference "#PWR047")
+					(reference "#PWR0150")
 					(unit 1)
 				)
@@
 		(dnp no)
 		(fields_autoplaced yes)
-		(property "Reference" "C19"
+		(property "Reference" "C18"
 			(at 114.3 77.4699 0)
 			(show_name no)
@@
 			(project "sd_hardware"
 				(path "/f972cb7f-90df-45d5-98d4-dc82335c3d91/898550ec-f46f-4748-8c3b-5dbafb3c9cde"
-					(reference "C19")
+					(reference "C18")
 					(unit 1)
 				)
@@
 		(dnp no)
 		(fields_autoplaced yes)
-		(property "Reference" "R40"
+		(property "Reference" "R37"
 			(at 96.52 77.4699 0)
 			(show_name no)
@@
 			(project "sd_hardware"
 				(path "/f972cb7f-90df-45d5-98d4-dc82335c3d91/898550ec-f46f-4748-8c3b-5dbafb3c9cde"
-					(reference "R40")
+					(reference "R37")
 					(unit 1)
 				)
@@
 		(dnp no)
 		(fields_autoplaced yes)
-		(property "Reference" "#PWR050"
+		(property "Reference" "#PWR0153"
 			(at 166.37 113.03 0)
 			(hide yes)
@@
 			(project "sd_hardware"
 				(path "/f972cb7f-90df-45d5-98d4-dc82335c3d91/898550ec-f46f-4748-8c3b-5dbafb3c9cde"
-					(reference "#PWR050")
-					(unit 1)
-				)
+					(reference "#PWR0153")
+					(unit 1)
+				)

Commit message: working
Other:
- title: (none) -> Solenoid_Driver_3.1 - Yamana
Changed lines of the file:
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@@
 	(generator_version "10.0")
 	(paper "A4")
+	(title_block
+		(title "Solenoid_Driver_3.1 - Yamana")
+		(date "2026-10-18")
+	)
 	(text "fail safe pull up to ¬CS"
 		(exclude_from_sim no)
