File: sd_hardware/Solenoid_Iso.kicad_sch (KiCad schematic)
At the start: 48 parts, among them IC10 TLP170AM_TPL,E, IC3 TLP170AM_TPL,E, IC4 TLP170AM_TPL,E, IC5 TLP170AM_TPL,E, IC6 TLP170AM_TPL,E, IC7 TLP170AM_TPL,E, IC8 TLP170AM_TPL,E, IC9 TLP170AM_TPL,E

Commit message: created schematic
Parts:
- D11: renamed from D33; footprint Diode_THT:Diode_Bridge_Round_D9.0mm -> Diode_SMD:D_SOD-323_HandSoldering
- D13: renamed from D25; footprint Diode_THT:Diode_Bridge_Round_D9.0mm -> Diode_SMD:D_SOD-323_HandSoldering
- D15: renamed from D31; footprint Diode_THT:Diode_Bridge_Round_D9.0mm -> Diode_SMD:D_SOD-323_HandSoldering
- D17: renamed from D27; footprint Diode_THT:Diode_Bridge_Round_D9.0mm -> Diode_SMD:D_SOD-323_HandSoldering
- D19: renamed from D29; footprint Diode_THT:Diode_Bridge_Round_D9.0mm -> Diode_SMD:D_SOD-323_HandSoldering
- D5: renamed from D20; footprint Diode_THT:Diode_Bridge_Round_D9.0mm -> Diode_SMD:D_SOD-323_HandSoldering
- D7: renamed from D35; footprint Diode_THT:Diode_Bridge_Round_D9.0mm -> Diode_SMD:D_SOD-323_HandSoldering
- D9: renamed from D23; footprint Diode_THT:Diode_Bridge_Round_D9.0mm -> Diode_SMD:D_SOD-323_HandSoldering
- IC2: renamed from IC3; footprint TLP170AMTPLE -> y-robo_footprint:TLP170AMTPLE
- IC3: renamed from IC4; footprint TLP170AMTPLE -> y-robo_footprint:TLP170AMTPLE
- IC4: renamed from IC5; footprint TLP170AMTPLE -> y-robo_footprint:TLP170AMTPLE
- IC5: renamed from IC6; footprint TLP170AMTPLE -> y-robo_footprint:TLP170AMTPLE
- IC6: renamed from IC7; footprint TLP170AMTPLE -> y-robo_footprint:TLP170AMTPLE
- IC7: renamed from IC8; footprint TLP170AMTPLE -> y-robo_footprint:TLP170AMTPLE
- IC8: renamed from IC9; footprint TLP170AMTPLE -> y-robo_footprint:TLP170AMTPLE
- IC9: renamed from IC10; footprint TLP170AMTPLE -> y-robo_footprint:TLP170AMTPLE
- R10: renamed from R14; footprint TLP170AMTPLE -> Resistor_SMD:R_0603_1608Metric_Pad0.98x0.95mm_HandSolder
- R11: renamed from R15; footprint TLP170AMTPLE -> Resistor_SMD:R_0603_1608Metric_Pad0.98x0.95mm_HandSolder
- R12: renamed from R16; footprint TLP170AMTPLE -> Resistor_SMD:R_0603_1608Metric_Pad0.98x0.95mm_HandSolder
- R13: renamed from R17; footprint TLP170AMTPLE -> Resistor_SMD:R_0603_1608Metric_Pad0.98x0.95mm_HandSolder
- R14: renamed from R18; footprint TLP170AMTPLE -> Resistor_SMD:R_0603_1608Metric_Pad0.98x0.95mm_HandSolder
- R15: renamed from R19; footprint TLP170AMTPLE -> Resistor_SMD:R_0603_1608Metric_Pad0.98x0.95mm_HandSolder
- R16: renamed from R20; footprint TLP170AMTPLE -> Resistor_SMD:R_0603_1608Metric_Pad0.98x0.95mm_HandSolder
- R23: renamed from R22; footprint TLP170AMTPLE -> Resistor_SMD:R_0603_1608Metric_Pad0.98x0.95mm_HandSolder
- R24: renamed from R23; footprint TLP170AMTPLE -> Resistor_SMD:R_0603_1608Metric_Pad0.98x0.95mm_HandSolder
- R25: renamed from R24; footprint TLP170AMTPLE -> Resistor_SMD:R_0603_1608Metric_Pad0.98x0.95mm_HandSolder
- R26: renamed from R25; footprint TLP170AMTPLE -> Resistor_SMD:R_0603_1608Metric_Pad0.98x0.95mm_HandSolder
- R27: renamed from R26; footprint TLP170AMTPLE -> Resistor_SMD:R_0603_1608Metric_Pad0.98x0.95mm_HandSolder
- R28: renamed from R27; footprint TLP170AMTPLE -> Resistor_SMD:R_0603_1608Metric_Pad0.98x0.95mm_HandSolder
- R29: renamed from R28; footprint TLP170AMTPLE -> Resistor_SMD:R_0603_1608Metric_Pad0.98x0.95mm_HandSolder
- R30: renamed from R29; footprint TLP170AMTPLE -> Resistor_SMD:R_0603_1608Metric_Pad0.98x0.95mm_HandSolder
- R9: renamed from R13; footprint TLP170AMTPLE -> Resistor_SMD:R_0603_1608Metric_Pad0.98x0.95mm_HandSolder
- renumbered D32 to D10, D24 to D12, D30 to D14, D26 to D16, D28 to D18, D21 to D4, D34 to D6, D22 to D8, R31 to R17, R36 to R18, R32 to R19, R35 to R20, R33 to R21, R34 to R22, R30 to R7, R37 to R8

Commit message: working
Parts:
- R1: renamed from R7; value 1.5k -> 3.3k
- R2: renamed from R8; value 1.5k -> 3.3k
- R3: renamed from R17; value 1.5k -> 3.3k
- R4: renamed from R18; value 1.5k -> 3.3k
- R5: renamed from R19; value 1.5k -> 3.3k
- R6: renamed from R20; value 1.5k -> 3.3k
- R7: renamed from R21; value 1.5k -> 3.3k
- R8: renamed from R22; value 1.5k -> 3.3k
- renumbered D5 to D1, D6 to D10, D8 to D11, D10 to D12, D12 to D13, D16 to D15, D18 to D16, D7 to D2, D9 to D3, D11 to D4, D13 to D5, D15 to D6, D17 to D7, D19 to D8, D4 to D9, IC2 to IC1, IC3 to IC2, IC4 to IC3, IC5 to IC4, IC6 to IC5, IC7 to IC6, IC8 to IC7, IC9 to IC8, R30 to R17, R29 to R18, R28 to R19, R27 to R20, R26 to R21, R25 to R22, R24 to R23, R23 to R24
Connections:
- net Solenoid2_-: no longer IC5.6 (D2)
- net Solenoid3_-: now also IC3.6 (D2); no longer IC2.6 (D2)
- net Solenoid4_-: now also IC4.6 (D2); no longer IC6.6 (D2)
- net Solenoid5_-: now also IC5.6 (D2); no longer IC3.6 (D2)
- net Solenoid6_-: now also IC6.6 (D2); no longer IC7.6 (D2)
- net Solenoid7_-: now also IC7.6 (D2); no longer IC4.6 (D2)
- new net PhotoRelay2_Drain: IC2.6 (D2)

Commit message: working
Connections:
- net PhotoRelay2_Drain is gone; now on net Solenoid2_-: IC2.6 (D2)

Commit message: working
Other:
- title: (none) -> Solenoid_Driver_3.1 - Yamana
Changed lines of the file:
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@@
 	(generator_version "10.0")
 	(paper "A4")
+	(title_block
+		(title "Solenoid_Driver_3.1 - Yamana")
+		(date "2026-10-18")
+	)
