File: sd_hardware/FDCAN_Transceiver.kicad_sch (KiCad schematic)
At the start: 3 parts, among them IC2 TJA1441AT

Commit message: fix
Parts:
- C15, C16: footprint Capacitor_SMD:C_0603_1608Metric -> Capacitor_SMD:C_0603_1608Metric_Pad1.08x0.95mm_HandSolder
- IC1: renamed from IC2; footprint TJA1441AT:SOIC127P600X175-8N -> y-robo_footprint:SOIC127P600X175-8N
Changed lines of the file:
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@@
 			)
 		)
-		(property "Footprint" "Capacitor_SMD:C_0603_1608Metric"
+		(property "Footprint" "Capacitor_SMD:C_0603_1608Metric_Pad1.08x0.95mm_HandSolder"
 			(at 117.8052 82.55 0)
 			(hide yes)
@@
 		(dnp no)
 		(fields_autoplaced yes)
-		(property "Reference" "#PWR040"
+		(property "Reference" "#PWR019"
 			(at 165.1 91.44 0)
 			(hide yes)
@@
 			(project "sd_hardware"
 				(path "/f972cb7f-90df-45d5-98d4-dc82335c3d91/7b080080-f198-43cb-b1ed-cfcaabba3163"
-					(reference "#PWR040")
+					(reference "#PWR019")
 					(unit 1)
 				)
@@
 		(in_pos_files yes)
 		(dnp no)
-		(property "Reference" "#PWR038"
+		(property "Reference" "#PWR017"
 			(at 116.84 54.61 0)
 			(hide yes)
@@
 			(project "sd_hardware"
 				(path "/f972cb7f-90df-45d5-98d4-dc82335c3d91/7b080080-f198-43cb-b1ed-cfcaabba3163"
-					(reference "#PWR038")
+					(reference "#PWR017")
 					(unit 1)
 				)
@@
 		(in_pos_files yes)
 		(dnp no)
-		(property "Reference" "#PWR039"
+		(property "Reference" "#PWR018"
 			(at 152.4 60.96 0)
 			(hide yes)
@@
 			(project "sd_hardware"
 				(path "/f972cb7f-90df-45d5-98d4-dc82335c3d91/7b080080-f198-43cb-b1ed-cfcaabba3163"
-					(reference "#PWR039")
+					(reference "#PWR018")
 					(unit 1)
 				)
@@
 			)
 		)
-		(property "Footprint" "Capacitor_SMD:C_0603_1608Metric"
+		(property "Footprint" "Capacitor_SMD:C_0603_1608Metric_Pad1.08x0.95mm_HandSolder"
 			(at 153.3652 82.55 0)
 			(hide yes)
@@
 		(dnp no)
 		(fields_autoplaced yes)
-		(property "Reference" "IC2"
+		(property "Reference" "IC1"
 			(at 137.16 57.15 0)
 			(show_name no)
@@
 			)
 		)
-		(property "Footprint" "TJA1441AT:SOIC127P600X175-8N"
+		(property "Footprint" "y-robo_footprint:SOIC127P600X175-8N"
 			(at 147.32 62.23 0)
 			(hide yes)
@@
 			(project "sd_hardware"
 				(path "/f972cb7f-90df-45d5-98d4-dc82335c3d91/7b080080-f198-43cb-b1ed-cfcaabba3163"
-					(reference "IC2")
-					(unit 1)
-				)
+					(reference "IC1")
+					(unit 1)
+				)

Commit message: fix var3.0 sd_hardware
Parts:
- renumbered IC1 to IC2
Changed lines of the file:
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@@
 		(dnp no)
 		(fields_autoplaced yes)
-		(property "Reference" "IC1"
+		(property "Reference" "IC2"
 			(at 137.16 57.15 0)
 			(show_name no)
@@
 			(project "sd_hardware"
 				(path "/f972cb7f-90df-45d5-98d4-dc82335c3d91/7b080080-f198-43cb-b1ed-cfcaabba3163"
-					(reference "IC1")
+					(reference "IC2")
 					(unit 1)
 				)

Commit message: created schematic
Parts:
- renumbered C15 to C14, C16 to C15, IC2 to IC10
Changed lines of the file:
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@@
 		(in_pos_files yes)
 		(dnp no)
-		(property "Reference" "C15"
+		(property "Reference" "C14"
 			(at 113.792 76.454 0)
 			(show_name no)
@@
 			(project "sd_hardware"
 				(path "/f972cb7f-90df-45d5-98d4-dc82335c3d91/7b080080-f198-43cb-b1ed-cfcaabba3163"
-					(reference "C15")
+					(reference "C14")
 					(unit 1)
 				)
@@
 		(dnp no)
 		(fields_autoplaced yes)
-		(property "Reference" "#PWR019"
+		(property "Reference" "#PWR040"
 			(at 165.1 91.44 0)
 			(hide yes)
@@
 			(project "sd_hardware"
 				(path "/f972cb7f-90df-45d5-98d4-dc82335c3d91/7b080080-f198-43cb-b1ed-cfcaabba3163"
-					(reference "#PWR019")
+					(reference "#PWR040")
 					(unit 1)
 				)
@@
 		(in_pos_files yes)
 		(dnp no)
-		(property "Reference" "#PWR017"
+		(property "Reference" "#PWR038"
 			(at 116.84 54.61 0)
 			(hide yes)
@@
 			(project "sd_hardware"
 				(path "/f972cb7f-90df-45d5-98d4-dc82335c3d91/7b080080-f198-43cb-b1ed-cfcaabba3163"
-					(reference "#PWR017")
+					(reference "#PWR038")
 					(unit 1)
 				)
@@
 		(in_pos_files yes)
 		(dnp no)
-		(property "Reference" "#PWR018"
+		(property "Reference" "#PWR039"
 			(at 152.4 60.96 0)
 			(hide yes)
@@
 			(project "sd_hardware"
 				(path "/f972cb7f-90df-45d5-98d4-dc82335c3d91/7b080080-f198-43cb-b1ed-cfcaabba3163"
-					(reference "#PWR018")
+					(reference "#PWR039")
 					(unit 1)
 				)
@@
 		(in_pos_files yes)
 		(dnp no)
-		(property "Reference" "C16"
+		(property "Reference" "C15"
 			(at 148.082 76.454 0)
 			(show_name no)
@@
 			(project "sd_hardware"
 				(path "/f972cb7f-90df-45d5-98d4-dc82335c3d91/7b080080-f198-43cb-b1ed-cfcaabba3163"
-					(reference "C16")
+					(reference "C15")
 					(unit 1)
 				)
@@
 		(dnp no)
 		(fields_autoplaced yes)
-		(property "Reference" "IC2"
+		(property "Reference" "IC10"
 			(at 137.16 57.15 0)
 			(show_name no)
@@
 			(project "sd_hardware"
 				(path "/f972cb7f-90df-45d5-98d4-dc82335c3d91/7b080080-f198-43cb-b1ed-cfcaabba3163"
-					(reference "IC2")
-					(unit 1)
-				)
+					(reference "IC10")
+					(unit 1)
+				)

Commit message: working
Parts:
- renumbered C14 to C16, C15 to C17
Changed lines of the file:
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@@
 		(in_pos_files yes)
 		(dnp no)
-		(property "Reference" "C14"
+		(property "Reference" "C16"
 			(at 113.792 76.454 0)
 			(show_name no)
@@
 			(project "sd_hardware"
 				(path "/f972cb7f-90df-45d5-98d4-dc82335c3d91/7b080080-f198-43cb-b1ed-cfcaabba3163"
-					(reference "C14")
+					(reference "C16")
 					(unit 1)
 				)
@@
 		(dnp no)
 		(fields_autoplaced yes)
-		(property "Reference" "#PWR040"
+		(property "Reference" "#PWR0143"
 			(at 165.1 91.44 0)
 			(hide yes)
@@
 			(project "sd_hardware"
 				(path "/f972cb7f-90df-45d5-98d4-dc82335c3d91/7b080080-f198-43cb-b1ed-cfcaabba3163"
-					(reference "#PWR040")
+					(reference "#PWR0143")
 					(unit 1)
 				)
@@
 		(in_pos_files yes)
 		(dnp no)
-		(property "Reference" "#PWR038"
+		(property "Reference" "#PWR0141"
 			(at 116.84 54.61 0)
 			(hide yes)
@@
 			(project "sd_hardware"
 				(path "/f972cb7f-90df-45d5-98d4-dc82335c3d91/7b080080-f198-43cb-b1ed-cfcaabba3163"
-					(reference "#PWR038")
+					(reference "#PWR0141")
 					(unit 1)
 				)
@@
 		(in_pos_files yes)
 		(dnp no)
-		(property "Reference" "#PWR039"
+		(property "Reference" "#PWR0142"
 			(at 152.4 60.96 0)
 			(hide yes)
@@
 			(project "sd_hardware"
 				(path "/f972cb7f-90df-45d5-98d4-dc82335c3d91/7b080080-f198-43cb-b1ed-cfcaabba3163"
-					(reference "#PWR039")
+					(reference "#PWR0142")
 					(unit 1)
 				)
@@
 		(in_pos_files yes)
 		(dnp no)
-		(property "Reference" "C15"
+		(property "Reference" "C17"
 			(at 148.082 76.454 0)
 			(show_name no)
@@
 			(project "sd_hardware"
 				(path "/f972cb7f-90df-45d5-98d4-dc82335c3d91/7b080080-f198-43cb-b1ed-cfcaabba3163"
-					(reference "C15")
-					(unit 1)
-				)
+					(reference "C17")
+					(unit 1)
+				)

Commit message: working
Other:
- title: (none) -> Solenoid_Driver_3.1 - Yamana
Changed lines of the file:
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@@
 	(generator_version "10.0")
 	(paper "A4")
+	(title_block
+		(title "Solenoid_Driver_3.1 - Yamana")
+		(date "2026-10-18")
+	)
 	(junction
 		(at 152.4 72.39)

Commit message: working
Parts:
- C17: value 0.1u -> 0.1μ
Changed lines of the file:
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@@
 			)
 		)
-		(property "Value" "0.1u"
+		(property "Value" "0.1μ"
 			(at 152.654 81.026 0)
 			(show_name no)
