File: sd_hardware/MCU_stm32_g431k8t6.kicad_sch (KiCad schematic)
At the start: 9 parts, among them J1 STLink-v3mini, SW1 SW_Push, U9 STM32G431K8Tx

Commit message: fix
Parts:
- C1: renamed from C9; footprint (none) -> Capacitor_SMD:C_0603_1608Metric_Pad1.08x0.95mm_HandSolder
- C2: renamed from C10; footprint (none) -> Capacitor_SMD:C_0603_1608Metric_Pad1.08x0.95mm_HandSolder
- C3: renamed from C11; footprint (none) -> Capacitor_SMD:C_0603_1608Metric_Pad1.08x0.95mm_HandSolder
- C4: renamed from C12; footprint (none) -> Capacitor_SMD:C_0603_1608Metric_Pad1.08x0.95mm_HandSolder
- C5: renamed from C13; footprint (none) -> Capacitor_SMD:C_0603_1608Metric_Pad1.08x0.95mm_HandSolder
- C6: renamed from C14; footprint (none) -> Capacitor_SMD:C_0603_1608Metric_Pad1.08x0.95mm_HandSolder
- J301: renamed from J1; footprint (none) -> y-robo_footprint:CONN14_3220-14_CNC
- SW301: renamed from SW1; footprint (none) -> y-robo_footprint:TVAF06-A020B-R
- renumbered U9 to U301
Connections:
- net ID_SW_BIT1: now also U301.29 (PB6); no longer U301.27 (PB4)
- net ID_SW_BIT3: now also U301.27 (PB4); no longer U301.29 (PB6)
- no-connect marks 6 -> 12
Changed lines of the file:
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@@
+	)
+	(no_connect
+		(at 43.18 63.5)
 	)
 	(no_connect
@@
 	)
 	(no_connect
+		(at 68.58 60.96)
+	)
+	(no_connect
 		(at 114.3 67.31)
 	)
@@
 	)
 	(no_connect
+		(at 68.58 63.5)
+	)
+	(no_connect
+		(at 68.58 76.2)
+	)
+	(no_connect
 		(at 127 72.39)
+	)
+	(no_connect
+		(at 68.58 58.42)
+	)
+	(no_connect
+		(at 43.18 50.8)
 	)
 	(wire
@@
 	(hierarchical_label "ID_SW_BIT3"
 		(shape input)
-		(at 43.18 60.96 180)
+		(at 43.18 55.88 180)
 		(effects
 			(font
@@
 	(hierarchical_label "ID_SW_BIT1"
 		(shape input)
-		(at 43.18 55.88 180)
+		(at 43.18 60.96 180)
 		(effects
 			(font
@@
 		(dnp no)
 		(fields_autoplaced yes)
-		(property "Reference" "J1"
+		(property "Reference" "J301"
 			(at 120.65 50.8 0)
 			(show_name no)
@@
 			)
 		)
-		(property "Footprint" ""
+		(property "Footprint" "y-robo_footprint:CONN14_3220-14_CNC"
 			(at 119.38 64.77 0)
 			(hide yes)
@@
 			(project "sd_hardware"
 				(path "/f972cb7f-90df-45d5-98d4-dc82335c3d91/2ec78280-fc8d-4c02-978a-5a90a50c2791"
-					(reference "J1")
+					(reference "J301")
 					(unit 1)
 				)
@@
 		(dnp no)
 		(fields_autoplaced yes)
-		(property "Reference" "C12"
+		(property "Reference" "C4"
 			(at 151.13 31.7499 0)
 			(show_name no)
@@
 			)
 		)
-		(property "Footprint" ""
+		(property "Footprint" "Capacitor_SMD:C_0603_1608Metric_Pad1.08x0.95mm_HandSolder"
 			(at 148.2852 36.83 0)
 			(hide yes)
@@
 			(project "sd_hardware"
 				(path "/f972cb7f-90df-45d5-98d4-dc82335c3d91/2ec78280-fc8d-4c02-978a-5a90a50c2791"
-					(reference "C12")
+					(reference "C4")
 					(unit 1)
 				)
@@
 		(dnp no)
 		(fields_autoplaced yes)
-		(property "Reference" "C13"
+		(property "Reference" "C5"
 			(at 161.29 31.7499 0)
 			(show_name no)
@@
 			)
 		)
-		(property "Footprint" ""
+		(property "Footprint" "Capacitor_SMD:C_0603_1608Metric_Pad1.08x0.95mm_HandSolder"
 			(at 158.4452 36.83 0)
 			(hide yes)
@@
 			(project "sd_hardware"
 				(path "/f972cb7f-90df-45d5-98d4-dc82335c3d91/2ec78280-fc8d-4c02-978a-5a90a50c2791"
-					(reference "C13")
+					(reference "C5")
 					(unit 1)
 				)
@@
 		(dnp no)
 		(fields_autoplaced yes)
-		(property "Reference" "#PWR037"
+		(property "Reference" "#PWR0308"
 			(at 167.64 71.12 0)
 			(hide yes)
@@
 			(project "sd_hardware"
 				(path "/f972cb7f-90df-45d5-98d4-dc82335c3d91/2ec78280-fc8d-4c02-978a-5a90a50c2791"
-					(reference "#PWR037")
+					(reference "#PWR0308")
 					(unit 1)
 				)
@@
 		(in_pos_files yes)
 		(dnp no)
-		(property "Reference" "C14"
+		(property "Reference" "C6"
 			(at 163.576 55.118 0)
 			(show_name no)
@@
 			)
 		)
-		(property "Footprint" ""
+		(property "Footprint" "Capacitor_SMD:C_0603_1608Metric_Pad1.08x0.95mm_HandSolder"
 			(at 168.6052 60.96 0)
 			(hide yes)
@@
 			(project "sd_hardware"
 				(path "/f972cb7f-90df-45d5-98d4-dc82335c3d91/2ec78280-fc8d-4c02-978a-5a90a50c2791"
-					(reference "C14")
+					(reference "C6")
 					(unit 1)
 				)
@@
 		(dnp no)
 		(fields_autoplaced yes)
-		(property "Reference" "U9"
+		(property "Reference" "U301"
 			(at 60.5633 83.82 0)
 			(show_name no)
@@
 			(project "sd_hardware"
 				(path "/f972cb7f-90df-45d5-98d4-dc82335c3d91/2ec78280-fc8d-4c02-978a-5a90a50c2791"
-					(reference "U9")
+					(reference "U301")
 					(unit 1)
 				)
@@
 		(dnp no)
 		(fields_autoplaced yes)
-		(property "Reference" "#PWR036"
+		(property "Reference" "#PWR0306"
 			(at 167.64 45.72 0)
 			(hide yes)
@@
 			(project "sd_hardware"
 				(path "/f972cb7f-90df-45d5-98d4-dc82335c3d91/2ec78280-fc8d-4c02-978a-5a90a50c2791"
-					(reference "#PWR036")
+					(reference "#PWR0306")
 					(unit 1)
 				)
@@
 		(dnp no)
 		(fields_autoplaced yes)
-		(property "Reference" "#PWR032"
+		(property "Reference" "#PWR0302"
 			(at 116.84 30.48 0)
 			(hide yes)
@@
 			(project "sd_hardware"
 				(path "/f972cb7f-90df-45d5-98d4-dc82335c3d91/2ec78280-fc8d-4c02-978a-5a90a50c2791"
-					(reference "#PWR032")
+					(reference "#PWR0302")
 					(unit 1)
 				)
@@
 		(dnp no)
 		(fields_autoplaced yes)
-		(property "Reference" "#PWR029"
+		(property "Reference" "#PWR0301"
 			(at 97.79 30.48 0)
 			(hide yes)
@@
 			(project "sd_hardware"
 				(path "/f972cb7f-90df-45d5-98d4-dc82335c3d91/2ec78280-fc8d-4c02-978a-5a90a50c2791"
-					(reference "#PWR029")
+					(reference "#PWR0301")
 					(unit 1)
 				)
@@
 		(dnp no)
 		(fields_autoplaced yes)
-		(property "Reference" "#PWR035"
+		(property "Reference" "#PWR0303"
 			(at 144.78 30.48 0)
 			(hide yes)
@@
 			(project "sd_hardware"
 				(path "/f972cb7f-90df-45d5-98d4-dc82335c3d91/2ec78280-fc8d-4c02-978a-5a90a50c2791"
-					(reference "#PWR035")
+					(reference "#PWR0303")
 					(unit 1)
 				)
@@
 		(dnp no)
 		(fields_autoplaced yes)
-		(property "Reference" "C9"
+		(property "Reference" "C1"
 			(at 104.14 31.7499 0)
 			(show_name no)
@@
 			)
 		)
-		(property "Footprint" ""
+		(property "Footprint" "Capacitor_SMD:C_0603_1608Metric_Pad1.08x0.95mm_HandSolder"
 			(at 101.2952 36.83 0)
 			(hide yes)
@@
 			(project "sd_hardware"
 				(path "/f972cb7f-90df-45d5-98d4-dc82335c3d91/2ec78280-fc8d-4c02-978a-5a90a50c2791"
-					(reference "C9")
+					(reference "C1")
 					(unit 1)
 				)
@@
 		(dnp no)
 		(fields_autoplaced yes)
-		(property "Reference" "SW1"
+		(property "Reference" "SW301"
 			(at 156.21 55.8799 90)
 			(show_name no)
@@
 			)
 		)
-		(property "Footprint" ""
+		(property "Footprint" "y-robo_footprint:TVAF06-A020B-R"
 			(at 157.48 57.15 0)
 			(hide yes)
@@
 			(project "sd_hardware"
 				(path "/f972cb7f-90df-45d5-98d4-dc82335c3d91/2ec78280-fc8d-4c02-978a-5a90a50c2791"
-					(reference "SW1")
+					(reference "SW301")
 					(unit 1)
 				)
@@
 		(dnp no)
 		(fields_autoplaced yes)
-		(property "Reference" "#PWR031"
+		(property "Reference" "#PWR0304"
 			(at 110.49 45.72 0)
 			(hide yes)
@@
 			(project "sd_hardware"
 				(path "/f972cb7f-90df-45d5-98d4-dc82335c3d91/2ec78280-fc8d-4c02-978a-5a90a50c2791"
-					(reference "#PWR031")
+					(reference "#PWR0304")
 					(unit 1)
 				)
@@
 		(dnp no)
 		(fields_autoplaced yes)
-		(property "Reference" "#PWR033"
+		(property "Reference" "#PWR0309"
 			(at 139.7 81.28 0)
 			(hide yes)
@@
 			(project "sd_hardware"
 				(path "/f972cb7f-90df-45d5-98d4-dc82335c3d91/2ec78280-fc8d-4c02-978a-5a90a50c2791"
-					(reference "#PWR033")
+					(reference "#PWR0309")
 					(unit 1)
 				)
@@
 		(dnp no)
 		(fields_autoplaced yes)
-		(property "Reference" "C11"
+		(property "Reference" "C3"
 			(at 134.62 31.7499 0)
 			(show_name no)
@@
 			)
 		)
-		(property "Footprint" ""
+		(property "Footprint" "Capacitor_SMD:C_0603_1608Metric_Pad1.08x0.95mm_HandSolder"
 			(at 131.7752 36.83 0)
 			(hide yes)
@@
 			(project "sd_hardware"
 				(path "/f972cb7f-90df-45d5-98d4-dc82335c3d91/2ec78280-fc8d-4c02-978a-5a90a50c2791"
-					(reference "C11")
+					(reference "C3")
 					(unit 1)
 				)
@@
 		(dnp no)
 		(fields_autoplaced yes)
-		(property "Reference" "C10"
+		(property "Reference" "C2"
 			(at 123.19 31.7499 0)
 			(show_name no)
@@
 			)
 		)
-		(property "Footprint" ""
+		(property "Footprint" "Capacitor_SMD:C_0603_1608Metric_Pad1.08x0.95mm_HandSolder"
 			(at 120.3452 36.83 0)
 			(hide yes)
@@
 			(project "sd_hardware"
 				(path "/f972cb7f-90df-45d5-98d4-dc82335c3d91/2ec78280-fc8d-4c02-978a-5a90a50c2791"
-					(reference "C10")
+					(reference "C2")
 					(unit 1)
 				)
@@
 		(dnp no)
 		(fields_autoplaced yes)
-		(property "Reference" "#PWR030"
+		(property "Reference" "#PWR0307"
 			(at 109.22 58.42 0)
 			(hide yes)
@@
 			(project "sd_hardware"
 				(path "/f972cb7f-90df-45d5-98d4-dc82335c3d91/2ec78280-fc8d-4c02-978a-5a90a50c2791"
-					(reference "#PWR030")
+					(reference "#PWR0307")
 					(unit 1)
 				)
@@
 		(dnp no)
 		(fields_autoplaced yes)
-		(property "Reference" "#PWR034"
+		(property "Reference" "#PWR0305"
 			(at 139.7 45.72 0)
 			(hide yes)
@@
 			(project "sd_hardware"
 				(path "/f972cb7f-90df-45d5-98d4-dc82335c3d91/2ec78280-fc8d-4c02-978a-5a90a50c2791"
-					(reference "#PWR034")
-					(unit 1)
-				)
+					(reference "#PWR0305")
+					(unit 1)
+				)

Commit message: fix var3.0 sd_hardware
Parts:
- added R21: 10k, Resistor_SMD:R_0603_1608Metric_Pad0.98x0.95mm_HandSolder, symbol Device:R
- renumbered J301 to J13, SW301 to SW1, U301 to U9
Connections:
- net BOOT0: now also R21.1
- net GND: now also R21.2
- net JTCK_SWCLK: now also U9.24 (PA14); no longer U9.23 (PA13)
- net JTMS_SWDIO: now also U9.23 (PA13); no longer U9.24 (PA14)
Changed lines of the file:
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@@
+	(wire
+		(pts
+			(xy 20.32 71.12) (xy 27.94 71.12)
+		)
+		(stroke
+			(width 0)
+			(type default)
+		)
+	)
 	(wire
 		(pts
@@
 	(wire
 		(pts
+			(xy 27.94 81.28) (xy 27.94 83.82)
+		)
+		(stroke
+			(width 0)
+			(type default)
+		)
+	)
+	(wire
+		(pts
 			(xy 167.64 63.5) (xy 167.64 64.77)
 		)
@@
 		(pts
 			(xy 111.76 69.85) (xy 111.76 74.93)
+		)
+		(stroke
+			(width 0)
+			(type default)
+		)
+	)
+	(wire
+		(pts
+			(xy 27.94 71.12) (xy 27.94 73.66)
 		)
 		(stroke
@@
 		)
 	)
+	(label "JTCK_SWCLK"
+		(at 93.98 73.66 180)
+		(effects
+			(font
+				(size 1.27 1.27)
+			)
+			(justify right bottom)
+		)
+	)
 	(label "VDD"
 		(at 139.7 27.94 180)
@@
 		)
 	)
-	(label "JTCK_SWCLK"
-		(at 93.98 71.12 180)
-		(effects
-			(font
-				(size 1.27 1.27)
-			)
-			(justify right bottom)
-		)
-	)
 	(label "JTDO_SWO"
 		(at 20.32 53.34 0)
@@
 		)
 	)
+	(label "BOOT0"
+		(at 20.32 71.12 0)
+		(effects
+			(font
+				(size 1.27 1.27)
+			)
+			(justify left bottom)
+		)
+	)
+	(label "JTMS_SWDIO"
+		(at 93.98 71.12 180)
+		(effects
+			(font
+				(size 1.27 1.27)
+			)
+			(justify right bottom)
+		)
+	)
 	(label "VSSA"
 		(at 58.42 90.17 90)
@@
 	(label "JTCK_SWCLK"
 		(at 139.7 62.23 180)
-		(effects
-			(font
-				(size 1.27 1.27)
-			)
-			(justify right bottom)
-		)
-	)
-	(label "JTMS_SWDIO"
-		(at 93.98 73.66 180)
 		(effects
 			(font
@@
 		(dnp no)
 		(fields_autoplaced yes)
-		(property "Reference" "J301"
+		(property "Reference" "J13"
 			(at 120.65 50.8 0)
 			(show_name no)
@@
 			(project "sd_hardware"
 				(path "/f972cb7f-90df-45d5-98d4-dc82335c3d91/2ec78280-fc8d-4c02-978a-5a90a50c2791"
-					(reference "J301")
+					(reference "J13")
 					(unit 1)
 				)
@@
 		(dnp no)
 		(fields_autoplaced yes)
-		(property "Reference" "U301"
+		(property "Reference" "U9"
 			(at 60.5633 83.82 0)
 			(show_name no)
@@
 			(project "sd_hardware"
 				(path "/f972cb7f-90df-45d5-98d4-dc82335c3d91/2ec78280-fc8d-4c02-978a-5a90a50c2791"
-					(reference "U301")
+					(reference "U9")
 					(unit 1)
 				)
@@
 	)
 	(symbol
+		(lib_id "Device:R")
+		(at 27.94 77.47 0)
+		(unit 1)
+		(body_style 1)
+		(exclude_from_sim no)
+		(in_bom yes)
+		(on_board yes)
+		(in_pos_files yes)
+		(dnp no)
+		(fields_autoplaced yes)
+		(property "Reference" "R21"
+			(at 30.48 76.1999 0)
+			(show_name no)
+			(do_not_autoplace no)
+			(effects
+				(font
+					(size 1.27 1.27)
+				)
+				(justify left)
+			)
+		)
+		(property "Value" "10k"
+			(at 30.48 78.7399 0)
+			(show_name no)
+			(do_not_autoplace no)
+			(effects
+				(font
+					(size 1.27 1.27)
+				)
+				(justify left)
+			)
+		)
+		(property "Footprint" "Resistor_SMD:R_0603_1608Metric_Pad0.98x0.95mm_HandSolder"
+			(at 26.162 77.47 90)
+			(hide yes)
+			(show_name no)
+			(do_not_autoplace no)
+			(effects
+				(font
+					(size 1.27 1.27)
+				)
+			)
+		)
+		(property "Datasheet" ""
+			(at 27.94 77.47 0)
+			(hide yes)
+			(show_name no)
+			(do_not_autoplace no)
+			(effects
+				(font
+					(size 1.27 1.27)
+				)
+			)
+		)
+		(property "Description" "Resistor"
+			(at 27.94 77.47 0)
+			(hide yes)
+			(show_name no)
+			(do_not_autoplace no)
+			(effects
+				(font
+					(size 1.27 1.27)
+				)
+			)
+		)
+		(pin "2"
+		)
+		(pin "1"
+		)
+		(instances
+			(project "sd_hardware"
+				(path "/f972cb7f-90df-45d5-98d4-dc82335c3d91/2ec78280-fc8d-4c02-978a-5a90a50c2791"
+					(reference "R21")
+					(unit 1)
+				)
+			)
+		)
+	)
+	(symbol
 		(lib_id "power:+3.3V")
 		(at 144.78 26.67 0)
@@
 	)
 	(symbol
+		(lib_id "power:GND")
+		(at 27.94 83.82 0)
+		(unit 1)
+		(body_style 1)
+		(exclude_from_sim no)
+		(in_bom yes)
+		(on_board yes)
+		(in_pos_files yes)
+		(dnp no)
+		(fields_autoplaced yes)
+		(property "Reference" "#PWR020"
+			(at 27.94 90.17 0)
+			(hide yes)
+			(show_name no)
+			(do_not_autoplace no)
+			(effects
+				(font
+					(size 1.27 1.27)
+				)
+			)
+		)
+		(property "Value" "GND"
+			(at 27.94 88.9 0)
+			(show_name no)
+			(do_not_autoplace no)
+			(effects
+				(font
+					(size 1.27 1.27)
+				)
+			)
+		)
+		(property "Footprint" ""
+			(at 27.94 83.82 0)
+			(hide yes)
+			(show_name no)
+			(do_not_autoplace no)
+			(effects
+				(font
+					(size 1.27 1.27)
+				)
+			)
+		)
+		(property "Datasheet" ""
+			(at 27.94 83.82 0)
+			(hide yes)
+			(show_name no)
+			(do_not_autoplace no)
+			(effects
+				(font
+					(size 1.27 1.27)
+				)
+			)
+		)
+		(property "Description" "Power symbol creates a global label with name \"GND\" , ground"
+			(at 27.94 83.82 0)
+			(hide yes)
+			(show_name no)
+			(do_not_autoplace no)
+			(effects
+				(font
+					(size 1.27 1.27)
+				)
+			)
+		)
+		(pin "1"
+		)
+		(instances
+			(project "sd_hardware"
+				(path "/f972cb7f-90df-45d5-98d4-dc82335c3d91/2ec78280-fc8d-4c02-978a-5a90a50c2791"
+					(reference "#PWR020")
+					(unit 1)
+				)
+			)
+		)
+	)
+	(symbol
 		(lib_id "Switch:SW_Push")
 		(at 152.4 57.15 270)
@@
 		(dnp no)
 		(fields_autoplaced yes)
-		(property "Reference" "SW301"
+		(property "Reference" "SW1"
 			(at 156.21 55.8799 90)
 			(show_name no)
@@
 			(project "sd_hardware"
 				(path "/f972cb7f-90df-45d5-98d4-dc82335c3d91/2ec78280-fc8d-4c02-978a-5a90a50c2791"
-					(reference "SW301")
-					(unit 1)
-				)
+					(reference "SW1")
+					(unit 1)
+				)

Commit message: delete RN
Other:
- moved on the sheet: R21
Changed lines of the file:
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@@
 	(wire
 		(pts
-			(xy 20.32 71.12) (xy 27.94 71.12)
+			(xy 106.68 83.82) (xy 114.3 83.82)
 		)
 		(stroke
@@
 	(wire
 		(pts
-			(xy 27.94 81.28) (xy 27.94 83.82)
+			(xy 114.3 93.98) (xy 114.3 96.52)
 		)
 		(stroke
@@
 	(wire
 		(pts
-			(xy 27.94 71.12) (xy 27.94 73.66)
+			(xy 114.3 83.82) (xy 114.3 86.36)
 		)
 		(stroke
@@
 	)
 	(label "BOOT0"
-		(at 20.32 71.12 0)
+		(at 106.68 83.82 0)
 		(effects
 			(font
@@
 	(symbol
 		(lib_id "Device:R")
-		(at 27.94 77.47 0)
+		(at 114.3 90.17 0)
 		(unit 1)
 		(body_style 1)
@@
 		(fields_autoplaced yes)
 		(property "Reference" "R21"
-			(at 30.48 76.1999 0)
+			(at 116.84 88.8999 0)
 			(show_name no)
 			(do_not_autoplace no)
@@
 		)
 		(property "Value" "10k"
-			(at 30.48 78.7399 0)
+			(at 116.84 91.4399 0)
 			(show_name no)
 			(do_not_autoplace no)
@@
 		)
 		(property "Footprint" "Resistor_SMD:R_0603_1608Metric_Pad0.98x0.95mm_HandSolder"
-			(at 26.162 77.47 90)
+			(at 112.522 90.17 90)
 			(hide yes)
 			(show_name no)
@@
 		)
 		(property "Datasheet" ""
-			(at 27.94 77.47 0)
+			(at 114.3 90.17 0)
 			(hide yes)
 			(show_name no)
@@
 		)
 		(property "Description" "Resistor"
-			(at 27.94 77.47 0)
+			(at 114.3 90.17 0)
 			(hide yes)
 			(show_name no)
@@
 	(symbol
 		(lib_id "power:GND")
-		(at 27.94 83.82 0)
+		(at 114.3 96.52 0)
 		(unit 1)
 		(body_style 1)
@@
 		(fields_autoplaced yes)
 		(property "Reference" "#PWR020"
-			(at 27.94 90.17 0)
+			(at 114.3 102.87 0)
 			(hide yes)
 			(show_name no)
@@
 		)
 		(property "Value" "GND"
-			(at 27.94 88.9 0)
+			(at 114.3 101.6 0)
 			(show_name no)
 			(do_not_autoplace no)
@@
 		)
 		(property "Footprint" ""
-			(at 27.94 83.82 0)
+			(at 114.3 96.52 0)
 			(hide yes)
 			(show_name no)
@@
 		)
 		(property "Datasheet" ""
-			(at 27.94 83.82 0)
+			(at 114.3 96.52 0)
 			(hide yes)
 			(show_name no)
@@
 		)
 		(property "Description" "Power symbol creates a global label with name \"GND\" , ground"
-			(at 27.94 83.82 0)
-			(hide yes)
-			(show_name no)
+			(at 114.3 96.52 0)
+			(hide yes)
+			(show_name no)
