File: sd_hardware/MCU_stm32_g431k8t6.kicad_sch (KiCad schematic)
At the start: 10 parts, among them J13 STLink-v3mini, SW1 SW_Push, U9 STM32G431K8Tx

Commit message: work
Connections:
- net ID_SW_BIT1: now also U9.18 (PA8); no longer U9.29 (PB6)
- net ID_SW_BIT2: now also U9.19 (PA9); no longer U9.28 (PB5)
- net ID_SW_BIT3: no longer U9.27 (PB4)
- net Solenoid1_GPIO: now also U9.27 (PB4); no longer U9.5 (PA0)
- net Solenoid2_GPIO: now also U9.28 (PB5); no longer U9.6 (PA1)
- net Solenoid3_GPIO: now also U9.29 (PB6); no longer U9.7 (PA2)
- net Solenoid4_GPIO: now also U9.30 (PB7); no longer U9.8 (PA3)
- net Solenoid5_GPIO: now also U9.5 (PA0); no longer U9.9 (PA4)
- net Solenoid6_GPIO: now also U9.6 (PA1); no longer U9.10 (PA5)
- net Solenoid7_GPIO: now also U9.7 (PA2); no longer U9.11 (PA6)
- net Solenoid8_GPIO: now also U9.8 (PA3); no longer U9.12 (PA7)
- net EP_Regu_LATCH: now reaches U9.13 (PB0)
- new net SPI1_MISO: U9.11 (PA6)
- new net SPI1_MOSI: U9.12 (PA7)
- new net SPI1_SCK: U9.10 (PA5)
- no-connect marks 12 -> 10
Changed lines of the file:
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@@
-	)
-	(no_connect
-		(at 43.18 63.5)
 	)
 	(no_connect
@@
 	)
 	(no_connect
+		(at 72.39 63.5)
+	)
+	(no_connect
 		(at 114.3 72.39)
-	)
-	(no_connect
-		(at 68.58 60.96)
 	)
 	(no_connect
@@
 	)
 	(no_connect
-		(at 68.58 63.5)
+		(at 68.58 76.2)
 	)
 	(no_connect
-		(at 68.58 76.2)
+		(at 68.58 48.26)
 	)
 	(no_connect
@@
 	)
 	(no_connect
-		(at 68.58 58.42)
-	)
-	(no_connect
-		(at 43.18 50.8)
+		(at 68.58 63.5)
 	)
 	(wire
@@
 	(wire
 		(pts
+			(xy 72.39 63.5) (xy 74.93 63.5)
+		)
+		(stroke
+			(width 0)
+			(type default)
+		)
+	)
+	(wire
+		(pts
 			(xy 119.38 38.1) (xy 130.81 38.1)
 		)
@@
 	(wire
 		(pts
-			(xy 20.32 53.34) (xy 43.18 53.34)
+			(xy 16.51 53.34) (xy 43.18 53.34)
 		)
 		(stroke
@@
 	(wire
 		(pts
-			(xy 20.32 66.04) (xy 43.18 66.04)
+			(xy 16.51 66.04) (xy 43.18 66.04)
 		)
 		(stroke
@@
 	)
 	(label "BOOT0"
-		(at 20.32 66.04 0)
+		(at 16.51 66.04 0)
 		(effects
 			(font
@@
 	)
 	(label "JTDO_SWO"
-		(at 20.32 53.34 0)
+		(at 16.51 53.34 0)
 		(effects
 			(font
@@
 		)
 	)
-	(hierarchical_label "Solenoid3_GPIO"
+	(hierarchical_label "Solenoid1_GPIO"
+		(shape output)
+		(at 43.18 55.88 180)
+		(effects
+			(font
+				(size 1.27 1.27)
+			)
+			(justify right)
+		)
+	)
+	(hierarchical_label "Solenoid4_GPIO"
+		(shape output)
+		(at 43.18 63.5 180)
+		(effects
+			(font
+				(size 1.27 1.27)
+			)
+			(justify right)
+		)
+	)
+	(hierarchical_label "Solenoid6_GPIO"
+		(shape output)
+		(at 68.58 40.64 0)
+		(effects
+			(font
+				(size 1.27 1.27)
+			)
+			(justify left)
+		)
+	)
+	(hierarchical_label "Solenoid2_GPIO"
+		(shape output)
+		(at 43.18 58.42 180)
+		(effects
+			(font
+				(size 1.27 1.27)
+			)
+			(justify right)
+		)
+	)
+	(hierarchical_label "EP_Regu_LATCH"
+		(shape output)
+		(at 43.18 50.8 180)
+		(effects
+			(font
+				(size 1.27 1.27)
+			)
+			(justify right)
+		)
+	)
+	(hierarchical_label "FDCAN1_TX"
+		(shape output)
+		(at 68.58 68.58 0)
+		(effects
+			(font
+				(size 1.27 1.27)
+			)
+			(justify left)
+		)
+	)
+	(hierarchical_label "Solenoid8_GPIO"
+		(shape output)
+		(at 68.58 45.72 0)
+		(effects
+			(font
+				(size 1.27 1.27)
+			)
+			(justify left)
+		)
+	)
+	(hierarchical_label "MCU_State_LED"
+		(shape output)
+		(at 43.18 43.18 180)
+		(effects
+			(font
+				(size 1.27 1.27)
+			)
+			(justify right)
+		)
+	)
+	(hierarchical_label "ID_SW_BIT3"
 		(shape input)
-		(at 68.58 43.18 0)
-		(effects
-			(font
-				(size 1.27 1.27)
-			)
-			(justify left)
-		)
-	)
-	(hierarchical_label "Solenoid7_GPIO"
+		(at 74.93 63.5 0)
+		(effects
+			(font
+				(size 1.27 1.27)
+			)
+			(justify left)
+		)
+	)
+	(hierarchical_label "SPI1_MISO"
 		(shape input)
 		(at 68.58 53.34 0)
@@
 			)
 			(justify left)
-		)
-	)
-	(hierarchical_label "Solenoid5_GPIO"
-		(shape input)
-		(at 68.58 48.26 0)
-		(effects
-			(font
-				(size 1.27 1.27)
-			)
-			(justify left)
-		)
-	)
-	(hierarchical_label "ID_SW_BIT3"
-		(shape input)
-		(at 43.18 55.88 180)
-		(effects
-			(font
-				(size 1.27 1.27)
-			)
-			(justify right)
-		)
-	)
-	(hierarchical_label "FDCAN1_LED"
-		(shape output)
-		(at 43.18 45.72 180)
-		(effects
-			(font
-				(size 1.27 1.27)
-			)
-			(justify right)
-		)
-	)
-	(hierarchical_label "Solenoid4_GPIO"
-		(shape input)
-		(at 68.58 45.72 0)
-		(effects
-			(font
-				(size 1.27 1.27)
-			)
-			(justify left)
-		)
-	)
-	(hierarchical_label "Solenoid2_GPIO"
-		(shape input)
-		(at 68.58 40.64 0)
-		(effects
-			(font
-				(size 1.27 1.27)
-			)
-			(justify left)
-		)
-	)
-	(hierarchical_label "Solenoid8_GPIO"
-		(shape input)
-		(at 68.58 55.88 0)
-		(effects
-			(font
-				(size 1.27 1.27)
-			)
-			(justify left)
-		)
-	)
-	(hierarchical_label "Solenoid6_GPIO"
-		(shape input)
-		(at 68.58 50.8 0)
-		(effects
-			(font
-				(size 1.27 1.27)
-			)
-			(justify left)
-		)
-	)
-	(hierarchical_label "Solenoid1_GPIO"
-		(shape input)
-		(at 68.58 38.1 0)
-		(effects
-			(font
-				(size 1.27 1.27)
-			)
-			(justify left)
-		)
-	)
-	(hierarchical_label "FDCAN1_TX"
-		(shape output)
-		(at 68.58 68.58 0)
-		(effects
-			(font
-				(size 1.27 1.27)
-			)
-			(justify left)
-		)
-	)
-	(hierarchical_label "ID_SW_BIT2"
-		(shape input)
-		(at 43.18 58.42 180)
-		(effects
-			(font
-				(size 1.27 1.27)
-			)
-			(justify right)
 		)
 	)
@@
 		)
 	)
-	(hierarchical_label "MCU_State_LED"
-		(shape output)
-		(at 43.18 43.18 180)
+	(hierarchical_label "SPI1_MOSI"
+		(shape output)
+		(at 68.58 55.88 0)
+		(effects
+			(font
+				(size 1.27 1.27)
+			)
+			(justify left)
+		)
+	)
+	(hierarchical_label "Solenoid7_GPIO"
+		(shape output)
+		(at 68.58 43.18 0)
+		(effects
+			(font
+				(size 1.27 1.27)
+			)
+			(justify left)
+		)
+	)
+	(hierarchical_label "Solenoid5_GPIO"
+		(shape output)
+		(at 68.58 38.1 0)
+		(effects
+			(font
+				(size 1.27 1.27)
+			)
+			(justify left)
+		)
+	)
+	(hierarchical_label "Solenoid3_GPIO"
+		(shape output)
+		(at 43.18 60.96 180)
+		(effects
+			(font
+				(size 1.27 1.27)
+			)
+			(justify right)
+		)
+	)
+	(hierarchical_label "FDCAN1_LED"
+		(shape output)
+		(at 43.18 45.72 180)
 		(effects
 			(font
@@
 	(hierarchical_label "ID_SW_BIT1"
 		(shape input)
-		(at 43.18 60.96 180)
-		(effects
-			(font
-				(size 1.27 1.27)
-			)
-			(justify right)
-		)
-	)
+		(at 68.58 58.42 0)
+		(effects
+			(font
+				(size 1.27 1.27)
+			)
+			(justify left)
+		)
+	)
+	(hierarchical_label "ID_SW_BIT2"
+		(shape input)
+		(at 68.58 60.96 0)
+		(effects
+			(font
+				(size 1.27 1.27)
+			)
+			(justify left)
+		)
+	)
+	(hierarchical_label "SPI1_SCK"
+		(shape output)
+		(at 68.58 50.8 0)
+		(effects
+			(font
+				(size 1.27 1.27)
+			)
+			(justify left)
+		)
+	)

Commit message: created schematic
Parts:
- renumbered C3 to C10, C4 to C11, C5 to C12, C6 to C13, C1 to C8, C2 to C9, J13 to J14, R21 to R31, SW1 to SW2, U9 to U1
Connections:
- net EP_Regu_ADC_CS: now reaches U1.9 (PA4)
- net EP_Regu_LATCH renamed EP_Regu_DAC_CS
- no-connect marks 10 -> 9
Changed lines of the file:
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@@
-	)
-	(no_connect
-		(at 68.58 48.26)
 	)
 	(no_connect
@@
 			)
 			(justify right bottom)
+		)
+	)
+	(hierarchical_label "EP_Regu_ADC_CS"
+		(shape output)
+		(at 68.58 48.26 0)
+		(effects
+			(font
+				(size 1.27 1.27)
+			)
+			(justify left)
 		)
 	)
@@
 		)
 	)
-	(hierarchical_label "EP_Regu_LATCH"
+	(hierarchical_label "EP_Regu_DAC_CS"
 		(shape output)
 		(at 43.18 50.8 180)
@@
 		(dnp no)
 		(fields_autoplaced yes)
-		(property "Reference" "J13"
+		(property "Reference" "J14"
 			(at 120.65 50.8 0)
 			(show_name no)
@@
 			(project "sd_hardware"
 				(path "/f972cb7f-90df-45d5-98d4-dc82335c3d91/2ec78280-fc8d-4c02-978a-5a90a50c2791"
-					(reference "J13")
+					(reference "J14")
 					(unit 1)
 				)
@@
 		(dnp no)
 		(fields_autoplaced yes)
-		(property "Reference" "C4"
+		(property "Reference" "C11"
 			(at 151.13 31.7499 0)
 			(show_name no)
@@
 			(project "sd_hardware"
 				(path "/f972cb7f-90df-45d5-98d4-dc82335c3d91/2ec78280-fc8d-4c02-978a-5a90a50c2791"
-					(reference "C4")
+					(reference "C11")
 					(unit 1)
 				)
@@
 		(dnp no)
 		(fields_autoplaced yes)
-		(property "Reference" "C5"
+		(property "Reference" "C12"
 			(at 161.29 31.7499 0)
 			(show_name no)
@@
 			(project "sd_hardware"
 				(path "/f972cb7f-90df-45d5-98d4-dc82335c3d91/2ec78280-fc8d-4c02-978a-5a90a50c2791"
-					(reference "C5")
+					(reference "C12")
 					(unit 1)
 				)
@@
 		(dnp no)
 		(fields_autoplaced yes)
-		(property "Reference" "#PWR0308"
+		(property "Reference" "#PWR035"
 			(at 167.64 71.12 0)
 			(hide yes)
@@
 			(project "sd_hardware"
 				(path "/f972cb7f-90df-45d5-98d4-dc82335c3d91/2ec78280-fc8d-4c02-978a-5a90a50c2791"
-					(reference "#PWR0308")
+					(reference "#PWR035")
 					(unit 1)
 				)
@@
 		(in_pos_files yes)
 		(dnp no)
-		(property "Reference" "C6"
+		(property "Reference" "C13"
 			(at 163.576 55.118 0)
 			(show_name no)
@@
 			(project "sd_hardware"
 				(path "/f972cb7f-90df-45d5-98d4-dc82335c3d91/2ec78280-fc8d-4c02-978a-5a90a50c2791"
-					(reference "C6")
+					(reference "C13")
 					(unit 1)
 				)
@@
 		(dnp no)
 		(fields_autoplaced yes)
-		(property "Reference" "U9"
+		(property "Reference" "U1"
 			(at 60.5633 83.82 0)
 			(show_name no)
@@
 			(project "sd_hardware"
 				(path "/f972cb7f-90df-45d5-98d4-dc82335c3d91/2ec78280-fc8d-4c02-978a-5a90a50c2791"
-					(reference "U9")
+					(reference "U1")
 					(unit 1)
 				)
@@
 		(dnp no)
 		(fields_autoplaced yes)
-		(property "Reference" "#PWR0306"
+		(property "Reference" "#PWR033"
 			(at 167.64 45.72 0)
 			(hide yes)
@@
 			(project "sd_hardware"
 				(path "/f972cb7f-90df-45d5-98d4-dc82335c3d91/2ec78280-fc8d-4c02-978a-5a90a50c2791"
-					(reference "#PWR0306")
+					(reference "#PWR033")
 					(unit 1)
 				)
@@
 		(dnp no)
 		(fields_autoplaced yes)
-		(property "Reference" "#PWR0302"
+		(property "Reference" "#PWR029"
 			(at 116.84 30.48 0)
 			(hide yes)
@@
 			(project "sd_hardware"
 				(path "/f972cb7f-90df-45d5-98d4-dc82335c3d91/2ec78280-fc8d-4c02-978a-5a90a50c2791"
-					(reference "#PWR0302")
+					(reference "#PWR029")
 					(unit 1)
 				)
@@
 		(dnp no)
 		(fields_autoplaced yes)
-		(property "Reference" "#PWR0301"
+		(property "Reference" "#PWR028"
 			(at 97.79 30.48 0)
 			(hide yes)
@@
 			(project "sd_hardware"
 				(path "/f972cb7f-90df-45d5-98d4-dc82335c3d91/2ec78280-fc8d-4c02-978a-5a90a50c2791"
-					(reference "#PWR0301")
+					(reference "#PWR028")
 					(unit 1)
 				)
@@
 		(dnp no)
 		(fields_autoplaced yes)
-		(property "Reference" "R21"
+		(property "Reference" "R31"
 			(at 116.84 88.8999 0)
 			(show_name no)
@@
 			(project "sd_hardware"
 				(path "/f972cb7f-90df-45d5-98d4-dc82335c3d91/2ec78280-fc8d-4c02-978a-5a90a50c2791"
-					(reference "R21")
+					(reference "R31")
 					(unit 1)
 				)
@@
 		(dnp no)
 		(fields_autoplaced yes)
-		(property "Reference" "#PWR0303"
+		(property "Reference" "#PWR030"
 			(at 144.78 30.48 0)
 			(hide yes)
@@
 			(project "sd_hardware"
 				(path "/f972cb7f-90df-45d5-98d4-dc82335c3d91/2ec78280-fc8d-4c02-978a-5a90a50c2791"
-					(reference "#PWR0303")
+					(reference "#PWR030")
 					(unit 1)
 				)
@@
 		(dnp no)
 		(fields_autoplaced yes)
-		(property "Reference" "C1"
+		(property "Reference" "C8"
 			(at 104.14 31.7499 0)
 			(show_name no)
@@
 			(project "sd_hardware"
 				(path "/f972cb7f-90df-45d5-98d4-dc82335c3d91/2ec78280-fc8d-4c02-978a-5a90a50c2791"
-					(reference "C1")
+					(reference "C8")
 					(unit 1)
 				)
@@
 		(dnp no)
 		(fields_autoplaced yes)
-		(property "Reference" "#PWR020"
+		(property "Reference" "#PWR037"
 			(at 114.3 102.87 0)
 			(hide yes)
@@
 			(project "sd_hardware"
 				(path "/f972cb7f-90df-45d5-98d4-dc82335c3d91/2ec78280-fc8d-4c02-978a-5a90a50c2791"
-					(reference "#PWR020")
+					(reference "#PWR037")
 					(unit 1)
 				)
@@
 		(dnp no)
 		(fields_autoplaced yes)
-		(property "Reference" "SW1"
+		(property "Reference" "SW2"
 			(at 156.21 55.8799 90)
 			(show_name no)
@@
 			(project "sd_hardware"
 				(path "/f972cb7f-90df-45d5-98d4-dc82335c3d91/2ec78280-fc8d-4c02-978a-5a90a50c2791"
-					(reference "SW1")
+					(reference "SW2")
 					(unit 1)
 				)
@@
 		(dnp no)
 		(fields_autoplaced yes)
-		(property "Reference" "#PWR0304"
+		(property "Reference" "#PWR031"
 			(at 110.49 45.72 0)
 			(hide yes)
@@
 			(project "sd_hardware"
 				(path "/f972cb7f-90df-45d5-98d4-dc82335c3d91/2ec78280-fc8d-4c02-978a-5a90a50c2791"
-					(reference "#PWR0304")
+					(reference "#PWR031")
 					(unit 1)
 				)
@@
 		(dnp no)
 		(fields_autoplaced yes)
-		(property "Reference" "#PWR0309"
+		(property "Reference" "#PWR036"
 			(at 139.7 81.28 0)
 			(hide yes)
@@
 			(project "sd_hardware"
 				(path "/f972cb7f-90df-45d5-98d4-dc82335c3d91/2ec78280-fc8d-4c02-978a-5a90a50c2791"
-					(reference "#PWR0309")
+					(reference "#PWR036")
 					(unit 1)
 				)
@@
 		(dnp no)
 		(fields_autoplaced yes)
-		(property "Reference" "C3"
+		(property "Reference" "C10"
 			(at 134.62 31.7499 0)
 			(show_name no)
@@
 			(project "sd_hardware"
 				(path "/f972cb7f-90df-45d5-98d4-dc82335c3d91/2ec78280-fc8d-4c02-978a-5a90a50c2791"
-					(reference "C3")
+					(reference "C10")
 					(unit 1)
 				)
@@
 		(dnp no)
 		(fields_autoplaced yes)
-		(property "Reference" "C2"
+		(property "Reference" "C9"
 			(at 123.19 31.7499 0)
 			(show_name no)
@@
 			(project "sd_hardware"
 				(path "/f972cb7f-90df-45d5-98d4-dc82335c3d91/2ec78280-fc8d-4c02-978a-5a90a50c2791"
-					(reference "C2")
+					(reference "C9")
 					(unit 1)
 				)
@@
 		(dnp no)
 		(fields_autoplaced yes)
-		(property "Reference" "#PWR0307"
+		(property "Reference" "#PWR034"
 			(at 109.22 58.42 0)
 			(hide yes)
@@
 			(project "sd_hardware"
 				(path "/f972cb7f-90df-45d5-98d4-dc82335c3d91/2ec78280-fc8d-4c02-978a-5a90a50c2791"
-					(reference "#PWR0307")
+					(reference "#PWR034")
 					(unit 1)
 				)
@@
 		(dnp no)
 		(fields_autoplaced yes)
-		(property "Reference" "#PWR0305"
+		(property "Reference" "#PWR032"
 			(at 139.7 45.72 0)
 			(hide yes)
@@
 			(project "sd_hardware"
 				(path "/f972cb7f-90df-45d5-98d4-dc82335c3d91/2ec78280-fc8d-4c02-978a-5a90a50c2791"
-					(reference "#PWR0305")
-					(unit 1)
-				)
+					(reference "#PWR032")
+					(unit 1)
+				)

Commit message: working
Parts:
- C1: renamed from C8; value 100n -> 0.1μ
- C2: renamed from C10; value 100n -> 0.1μ
- renumbered C13 to C3, C9 to C4, C11 to C5, C12 to C6, J14 to J9, R31 to R25, SW2 to SW1
Changed lines of the file:
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@@
 		(dnp no)
 		(fields_autoplaced yes)
-		(property "Reference" "J14"
+		(property "Reference" "J9"
 			(at 120.65 50.8 0)
 			(show_name no)
@@
 			(project "sd_hardware"
 				(path "/f972cb7f-90df-45d5-98d4-dc82335c3d91/2ec78280-fc8d-4c02-978a-5a90a50c2791"
-					(reference "J14")
+					(reference "J9")
 					(unit 1)
 				)
@@
 		(dnp no)
 		(fields_autoplaced yes)
-		(property "Reference" "C11"
+		(property "Reference" "C5"
 			(at 151.13 31.7499 0)
 			(show_name no)
@@
 			(project "sd_hardware"
 				(path "/f972cb7f-90df-45d5-98d4-dc82335c3d91/2ec78280-fc8d-4c02-978a-5a90a50c2791"
-					(reference "C11")
+					(reference "C5")
 					(unit 1)
 				)
@@
 		(dnp no)
 		(fields_autoplaced yes)
-		(property "Reference" "C12"
+		(property "Reference" "C6"
 			(at 161.29 31.7499 0)
 			(show_name no)
@@
 			(project "sd_hardware"
 				(path "/f972cb7f-90df-45d5-98d4-dc82335c3d91/2ec78280-fc8d-4c02-978a-5a90a50c2791"
-					(reference "C12")
+					(reference "C6")
 					(unit 1)
 				)
@@
 		(dnp no)
 		(fields_autoplaced yes)
-		(property "Reference" "#PWR035"
+		(property "Reference" "#PWR0138"
 			(at 167.64 71.12 0)
 			(hide yes)
@@
 			(project "sd_hardware"
 				(path "/f972cb7f-90df-45d5-98d4-dc82335c3d91/2ec78280-fc8d-4c02-978a-5a90a50c2791"
-					(reference "#PWR035")
+					(reference "#PWR0138")
 					(unit 1)
 				)
@@
 		(in_pos_files yes)
 		(dnp no)
-		(property "Reference" "C13"
+		(property "Reference" "C3"
 			(at 163.576 55.118 0)
 			(show_name no)
@@
 			(project "sd_hardware"
 				(path "/f972cb7f-90df-45d5-98d4-dc82335c3d91/2ec78280-fc8d-4c02-978a-5a90a50c2791"
-					(reference "C13")
+					(reference "C3")
 					(unit 1)
 				)
@@
 		(dnp no)
 		(fields_autoplaced yes)
-		(property "Reference" "#PWR033"
+		(property "Reference" "#PWR0136"
 			(at 167.64 45.72 0)
 			(hide yes)
@@
 			(project "sd_hardware"
 				(path "/f972cb7f-90df-45d5-98d4-dc82335c3d91/2ec78280-fc8d-4c02-978a-5a90a50c2791"
-					(reference "#PWR033")
+					(reference "#PWR0136")
 					(unit 1)
 				)
@@
 		(dnp no)
 		(fields_autoplaced yes)
-		(property "Reference" "#PWR029"
+		(property "Reference" "#PWR0132"
 			(at 116.84 30.48 0)
 			(hide yes)
@@
 			(project "sd_hardware"
 				(path "/f972cb7f-90df-45d5-98d4-dc82335c3d91/2ec78280-fc8d-4c02-978a-5a90a50c2791"
-					(reference "#PWR029")
+					(reference "#PWR0132")
 					(unit 1)
 				)
@@
 		(dnp no)
 		(fields_autoplaced yes)
-		(property "Reference" "#PWR028"
+		(property "Reference" "#PWR0131"
 			(at 97.79 30.48 0)
 			(hide yes)
@@
 			(project "sd_hardware"
 				(path "/f972cb7f-90df-45d5-98d4-dc82335c3d91/2ec78280-fc8d-4c02-978a-5a90a50c2791"
-					(reference "#PWR028")
+					(reference "#PWR0131")
 					(unit 1)
 				)
@@
 		(dnp no)
 		(fields_autoplaced yes)
-		(property "Reference" "R31"
+		(property "Reference" "R25"
 			(at 116.84 88.8999 0)
 			(show_name no)
@@
 			(project "sd_hardware"
 				(path "/f972cb7f-90df-45d5-98d4-dc82335c3d91/2ec78280-fc8d-4c02-978a-5a90a50c2791"
-					(reference "R31")
+					(reference "R25")
 					(unit 1)
 				)
@@
 		(dnp no)
 		(fields_autoplaced yes)
-		(property "Reference" "#PWR030"
+		(property "Reference" "#PWR0133"
 			(at 144.78 30.48 0)
 			(hide yes)
@@
 			(project "sd_hardware"
 				(path "/f972cb7f-90df-45d5-98d4-dc82335c3d91/2ec78280-fc8d-4c02-978a-5a90a50c2791"
-					(reference "#PWR030")
+					(reference "#PWR0133")
 					(unit 1)
 				)
@@
 		(dnp no)
 		(fields_autoplaced yes)
-		(property "Reference" "C8"
+		(property "Reference" "C1"
 			(at 104.14 31.7499 0)
 			(show_name no)
@@
 			)
 		)
-		(property "Value" "100n"
+		(property "Value" "0.1μ"
 			(at 104.14 34.2899 0)
 			(show_name no)
@@
 			(project "sd_hardware"
 				(path "/f972cb7f-90df-45d5-98d4-dc82335c3d91/2ec78280-fc8d-4c02-978a-5a90a50c2791"
-					(reference "C8")
+					(reference "C1")
 					(unit 1)
 				)
@@
 		(dnp no)
 		(fields_autoplaced yes)
-		(property "Reference" "#PWR037"
+		(property "Reference" "#PWR0140"
 			(at 114.3 102.87 0)
 			(hide yes)
@@
 			(project "sd_hardware"
 				(path "/f972cb7f-90df-45d5-98d4-dc82335c3d91/2ec78280-fc8d-4c02-978a-5a90a50c2791"
-					(reference "#PWR037")
+					(reference "#PWR0140")
 					(unit 1)
 				)
@@
 		(dnp no)
 		(fields_autoplaced yes)
-		(property "Reference" "SW2"
+		(property "Reference" "SW1"
 			(at 156.21 55.8799 90)
 			(show_name no)
@@
 			(project "sd_hardware"
 				(path "/f972cb7f-90df-45d5-98d4-dc82335c3d91/2ec78280-fc8d-4c02-978a-5a90a50c2791"
-					(reference "SW2")
+					(reference "SW1")
 					(unit 1)
 				)
@@
 		(dnp no)
 		(fields_autoplaced yes)
-		(property "Reference" "#PWR031"
+		(property "Reference" "#PWR0134"
 			(at 110.49 45.72 0)
 			(hide yes)
@@
 			(project "sd_hardware"
 				(path "/f972cb7f-90df-45d5-98d4-dc82335c3d91/2ec78280-fc8d-4c02-978a-5a90a50c2791"
-					(reference "#PWR031")
+					(reference "#PWR0134")
 					(unit 1)
 				)
@@
 		(dnp no)
 		(fields_autoplaced yes)
-		(property "Reference" "#PWR036"
+		(property "Reference" "#PWR0139"
 			(at 139.7 81.28 0)
 			(hide yes)
@@
 			(project "sd_hardware"
 				(path "/f972cb7f-90df-45d5-98d4-dc82335c3d91/2ec78280-fc8d-4c02-978a-5a90a50c2791"
-					(reference "#PWR036")
+					(reference "#PWR0139")
 					(unit 1)
 				)
@@
 		(dnp no)
 		(fields_autoplaced yes)
-		(property "Reference" "C10"
+		(property "Reference" "C2"
 			(at 134.62 31.7499 0)
 			(show_name no)
@@
 			)
 		)
-		(property "Value" "100n"
+		(property "Value" "0.1μ"
 			(at 134.62 34.2899 0)
 			(show_name no)
@@
 			(project "sd_hardware"
 				(path "/f972cb7f-90df-45d5-98d4-dc82335c3d91/2ec78280-fc8d-4c02-978a-5a90a50c2791"
-					(reference "C10")
+					(reference "C2")
 					(unit 1)
 				)
@@
 		(dnp no)
 		(fields_autoplaced yes)
-		(property "Reference" "C9"
+		(property "Reference" "C4"
 			(at 123.19 31.7499 0)
 			(show_name no)
@@
 			(project "sd_hardware"
 				(path "/f972cb7f-90df-45d5-98d4-dc82335c3d91/2ec78280-fc8d-4c02-978a-5a90a50c2791"
-					(reference "C9")
+					(reference "C4")
 					(unit 1)
 				)
@@
 		(dnp no)
 		(fields_autoplaced yes)
-		(property "Reference" "#PWR034"
+		(property "Reference" "#PWR0137"
 			(at 109.22 58.42 0)
 			(hide yes)
@@
 			(project "sd_hardware"
 				(path "/f972cb7f-90df-45d5-98d4-dc82335c3d91/2ec78280-fc8d-4c02-978a-5a90a50c2791"
-					(reference "#PWR034")
+					(reference "#PWR0137")
 					(unit 1)
 				)
@@
 		(dnp no)
 		(fields_autoplaced yes)
-		(property "Reference" "#PWR032"
+		(property "Reference" "#PWR0135"
 			(at 139.7 45.72 0)
 			(hide yes)
@@
 			(project "sd_hardware"
 				(path "/f972cb7f-90df-45d5-98d4-dc82335c3d91/2ec78280-fc8d-4c02-978a-5a90a50c2791"
-					(reference "#PWR032")
-					(unit 1)
-				)
+					(reference "#PWR0135")
+					(unit 1)
+				)

Commit message: working
Other:
- title: (none) -> Solenoid_Driver_3.1 - Yamana
Changed lines of the file:
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@@
 	(generator_version "10.0")
 	(paper "A4")
+	(title_block
+		(title "Solenoid_Driver_3.1 - Yamana")
+		(date "2026-10-18")
+	)
 	(text "Decoupling Capacitor\nVBAT: none\nVDD: 100nF*2 + 4.7μF\nVDDA: 10nF + 1μF\nVREF: none\n\nDatasheet 68p.\nhttps://www.st.com/resource/en/datasheet/DM00507199.pdf"
 		(exclude_from_sim no)

Commit message: working
Connections:
- net ID_SW_BIT3: now also U1.20 (PA10)
- no-connect marks 9 -> 7
Changed lines of the file:
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@@
-	)
-	(no_connect
-		(at 72.39 63.5)
 	)
 	(no_connect
@@
 		(at 127 72.39)
 	)
-	(no_connect
-		(at 68.58 63.5)
-	)
 	(wire
 		(pts
@@
 		(pts
 			(xy 111.76 64.77) (xy 114.3 64.77)
-		)
-		(stroke
-			(width 0)
-			(type default)
-		)
-	)
-	(wire
-		(pts
-			(xy 72.39 63.5) (xy 74.93 63.5)
 		)
 		(stroke
@@
 	(hierarchical_label "ID_SW_BIT3"
 		(shape input)
-		(at 74.93 63.5 0)
-		(effects
-			(font
+		(at 68.58 63.5 0)
+		(effects
+			(font
