File: sd_hardware/SPI_DAC.kicad_sch (KiCad schematic)
At the start: 0 parts

Commit message: created schematic
Parts:
- added C16: 0.1μ, Capacitor_SMD:C_0603_1608Metric_Pad1.08x0.95mm_HandSolder, symbol Device:C
- added C17: 1μ, Capacitor_SMD:C_0603_1608Metric_Pad1.08x0.95mm_HandSolder, symbol Device:C
- added C18: 220nF, Capacitor_SMD:C_0603_1608Metric_Pad1.08x0.95mm_HandSolder, symbol Device:C
- added R32, R33, R36, R38: 0, Resistor_SMD:R_0603_1608Metric_Pad0.98x0.95mm_HandSolder, symbol Device:R
- added R34, R35: 40k, Resistor_SMD:R_0603_1608Metric_Pad0.98x0.95mm_HandSolder, symbol Device:R
- added R37, R39: 10k, Resistor_SMD:R_0603_1608Metric_Pad0.98x0.95mm_HandSolder, symbol Device:R
- added U2: DAC60501ZDGSR, y-robo_footprint:DGS10_TEX, symbol DAC60501ZDGSR:DAC60501ZDGSR
- added U3: BD87521G-LB, y-robo_footprint:SOT95P280X125-5N, symbol y-robo:BD87521G-LB
Connections:
- new net: R32.2, R35.1, R36.1
- new net: C18.1, U2.10 (VREFIO)
- new net: R37.2, U2.2 (VOUT)
- new net: R33.2, R34.1, R38.1
- new net +12V: C16.1, C17.1, U3.5 (V+)
- new net +5VP: U2.1 (VDD)
- new net +VSENSE: R32.1
- new net -VSENSE: R33.1
- new net CS_N: U2.7 (*SYNC/A0)
- new net GND: C18.2, U2.4 (AGND), U2.5 (SPI2C)
- new net GNDPWR: C16.2, C17.2, R38.2, R39.1, U3.2 (V-)
- new net OP_VIN+: R34.2, R37.1, U3.3 (+)
- new net OP_VIN-: R35.2, R39.2, U3.4 (-)
- new net SCLK: U2.6 (SCLK/SCL)
- new net SDIN: U2.8 (SDIN/SDA)
- new net VOUT: R36.2, U3.1

Commit message: working
Parts:
- renumbered C16 to C20, C17 to C21, C18 to C22, R32 to R39, R33 to R40, R34 to R41, R35 to R42, R36 to R43, R37 to R44, R38 to R45, R39 to R46, U2 to U3, U3 to U4
Connections:
- net GND is gone; now on net GNDPWR: C22.2, U3.4 (AGND), U3.5 (SPI2C)

Commit message: working
Other:
- title: (none) -> Solenoid_Driver_3.1 - Yamana
- moved on the sheet: C20, C21
Changed lines of the file:
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@@
 	(generator_version "10.0")
 	(paper "A4")
+	(title_block
+		(title "Solenoid_Driver_3.1 - Yamana")
+		(date "2026-10-18")
+	)
 	(junction
 		(at 72.39 72.39)
@@
 	)
 	(junction
-		(at 90.17 53.34)
+		(at 85.09 53.34)
 		(diameter 0)
 		(color 0 0 0 0)
@@
 	)
 	(junction
-		(at 83.82 53.34)
+		(at 90.17 53.34)
 		(diameter 0)
 		(color 0 0 0 0)
@@
 	(wire
 		(pts
+			(xy 85.09 63.5) (xy 92.71 63.5)
+		)
+		(stroke
+			(width 0)
+			(type default)
+		)
+	)
+	(wire
+		(pts
 			(xy 185.42 80.01) (xy 199.39 80.01)
 		)
@@
 	(wire
 		(pts
-			(xy 83.82 53.34) (xy 83.82 54.61)
+			(xy 90.17 53.34) (xy 90.17 54.61)
 		)
 		(stroke
@@
 	(wire
 		(pts
-			(xy 90.17 53.34) (xy 97.79 53.34)
-		)
-		(stroke
-			(width 0)
-			(type default)
-		)
-	)
-	(wire
-		(pts
 			(xy 58.42 72.39) (xy 62.23 72.39)
 		)
@@
 	(wire
 		(pts
-			(xy 81.28 53.34) (xy 83.82 53.34)
+			(xy 81.28 53.34) (xy 97.79 53.34)
 		)
 		(stroke
@@
 	(wire
 		(pts
-			(xy 90.17 63.5) (xy 92.71 63.5)
-		)
-		(stroke
-			(width 0)
-			(type default)
-		)
-	)
-	(wire
-		(pts
 			(xy 199.39 92.71) (xy 199.39 93.98)
 		)
@@
 	(wire
 		(pts
-			(xy 83.82 63.5) (xy 90.17 63.5)
-		)
-		(stroke
-			(width 0)
-			(type default)
-		)
-	)
-	(wire
-		(pts
 			(xy 132.08 76.2) (xy 132.08 80.01)
 		)
@@
 	(wire
 		(pts
-			(xy 83.82 62.23) (xy 83.82 63.5)
-		)
-		(stroke
-			(width 0)
-			(type default)
-		)
-	)
-	(wire
-		(pts
-			(xy 83.82 53.34) (xy 90.17 53.34)
+			(xy 90.17 62.23) (xy 90.17 63.5)
 		)
 		(stroke
@@
 	(wire
 		(pts
-			(xy 90.17 62.23) (xy 90.17 63.5)
+			(xy 85.09 62.23) (xy 85.09 63.5)
 		)
 		(stroke
@@
 	(wire
 		(pts
-			(xy 90.17 53.34) (xy 90.17 54.61)
+			(xy 85.09 53.34) (xy 85.09 54.61)
 		)
 		(stroke
@@
 	(symbol
 		(lib_id "Device:C")
-		(at 90.17 58.42 0)
+		(at 85.09 58.42 0)
 		(unit 1)
 		(body_style 1)
@@
 		(dnp no)
 		(property "Reference" "C21"
-			(at 86.106 56.388 0)
+			(at 81.026 56.388 0)
 			(show_name no)
 			(do_not_autoplace no)
@@
 		)
 		(property "Value" "1μ"
-			(at 90.17 60.706 0)
+			(at 85.09 60.706 0)
 			(show_name no)
 			(do_not_autoplace no)
@@
 		)
 		(property "Footprint" "Capacitor_SMD:C_0603_1608Metric_Pad1.08x0.95mm_HandSolder"
-			(at 91.1352 62.23 0)
+			(at 86.0552 62.23 0)
 			(hide yes)
 			(show_name no)
@@
 		)
 		(property "Datasheet" ""
-			(at 90.17 58.42 0)
+			(at 85.09 58.42 0)
 			(hide yes)
 			(show_name no)
@@
 		)
 		(property "Description" "Unpolarized capacitor"
-			(at 90.17 58.42 0)
+			(at 85.09 58.42 0)
 			(hide yes)
 			(show_name no)
@@
 	(symbol
 		(lib_id "Device:C")
-		(at 83.82 58.42 0)
+		(at 90.17 58.42 0)
 		(unit 1)
 		(body_style 1)
@@
 		(dnp no)
 		(property "Reference" "C20"
-			(at 79.756 56.388 0)
+			(at 86.106 56.388 0)
 			(show_name no)
 			(do_not_autoplace no)
@@
 		)
 		(property "Value" "0.1μ"
-			(at 83.82 60.706 0)
+			(at 90.17 60.706 0)
 			(show_name no)
 			(do_not_autoplace no)
@@
 		)
 		(property "Footprint" "Capacitor_SMD:C_0603_1608Metric_Pad1.08x0.95mm_HandSolder"
-			(at 84.7852 62.23 0)
+			(at 91.1352 62.23 0)
 			(hide yes)
 			(show_name no)
@@
 		)
 		(property "Datasheet" ""
-			(at 83.82 58.42 0)
+			(at 90.17 58.42 0)
 			(hide yes)
 			(show_name no)
@@
 		)
 		(property "Description" "Unpolarized capacitor"
-			(at 83.82 58.42 0)
-			(hide yes)
-			(show_name no)
+			(at 90.17 58.42 0)
+			(hide yes)
+			(show_name no)

Commit message: working
Parts:
- removed R39, R40, R43, R45: 0, Resistor_SMD:R_0603_1608Metric_Pad0.98x0.95mm_HandSolder, symbol Device:R
- added C26: 1μ, Capacitor_SMD:C_0603_1608Metric_Pad1.08x0.95mm_HandSolder, symbol Device:C
- added C27: 0.1μ, Capacitor_SMD:C_0603_1608Metric_Pad1.08x0.95mm_HandSolder, symbol Device:C
- added JP3, JP4: SolderJumper_3_Open, Jumper:SolderJumper-3_P1.3mm_Open_RoundedPad1.0x1.5mm_NumberLabels, symbol Jumper:SolderJumper_3_Open
Connections:
- net +5VP: now also C26.1, C27.1
- net +VSENSE: now also JP3.3 (B)
- net -VSENSE: now also JP4.3 (B)
- net GNDPWR: now also C26.2, C27.2, JP4.1 (A)
- net VOUT: now also JP3.1 (A)
- net at R42.1: now also JP3.2 (C)
- net at R41.1: now also JP4.2 (C)
