File: sd_hardware/sd_hardware.kicad_pcb (KiCad board)
At the start: 2 copper layers, 95.5 x 61.8 mm, 135 parts, among them IC1 TLP170AM_TPL,E, IC10 TJA1441AT, IC2 TLP170AM_TPL,E, IC3 TLP170AM_TPL,E, IC4 TLP170AM_TPL,E, IC5 TLP170AM_TPL,E, IC6 TLP170AM_TPL,E, IC7 TLP170AM_TPL,E, IC8 TLP170AM_TPL,E, IC9 BD9E201FP4-Z, J1 Conn_01x02_Socket, J10 RJ45, J11 RJ45, J12 Conn_01x02_Socket, J13 XT60PW-M_1x02_Horizontal, J14 Conn_01x06_Socket, J2 Conn_01x02_Socket, J3 Conn_01x02_Socket, J4 Conn_01x02_Socket, J5 Conn_01x02_Socket, J6 Conn_01x02_Socket, J7 Conn_01x02_Socket, J8 Conn_01x02_Socket, J9 STLink-v3mini, SW1 SW_Push, SW2 SW_DIP_x03, U1 STM32G431K8Tx, U2 ADUM251N1BRIZ, U3 DAC60501ZDGSR, U4 BD87521G-LB, U5 BD87581YG-C, U6 ADS1018IDGSR, U7 BD00FC0WEFJ

Commit message: working
Parts:
- added J15: Conn_01x04_Socket, Connector_JST:JST_XH_B4B-XH-A_1x04_P2.50mm_Vertical, F.Cu at (137.8, 107.7)
- C11, C12: footprint Capacitor_SMD:C_0603_1608Metric_Pad1.08x0.95mm_HandSolder -> Capacitor_SMD:C_1210_3225Metric_Pad1.33x2.70mm_HandSolder
- moved C12 13.1 mm to (130.2, 83.8)
- moved C11 11.5 mm to (127.0, 83.8)
- moved R41 9.78 mm to (121.8, 97.2), turned to 0 degrees
- moved R54 9.78 mm to (142.2, 92.0)
- moved C18 9.75 mm to (158.5, 97.2)
- moved R28 9.72 mm to (162.2, 94.2)
- moved R29 9.72 mm to (162.2, 92.8)
- moved R30 9.72 mm to (162.2, 91.2)
- moved R31 9.72 mm to (162.2, 90.2)
- moved R37 9.72 mm to (162.2, 94.2)
- moved R38 9.72 mm to (162.2, 92.8)
- moved R52 9.72 mm to (162.2, 88.8)
- moved R53 9.53 mm to (142.2, 90.2), turned to 0 degrees
- moved C19 9.50 mm to (145.0, 97.2)
- moved U2 9.50 mm to (151.2, 91.0)
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Connections:
- U2 pad 12: /SPI_ADC/MOSI -> /SPI_Iso/MOSI_OUT
- U2 pad 13: /SPI_ADC/SCLK -> /SPI_Iso/CLK_OUT
- U2 pad 6: /MCU_stm32_g431k8t6/SPI1_MISO -> /SPI_Iso/MISO_OUT
Routing:
- net +12V: track 173.6 -> 253.2 mm, vias 1 -> 3
- net +5VP: track 2.89 -> 68.3 mm, vias 0 -> 2
- net +3.3V: track 78.2 -> 136.4 mm, vias 2 -> 4
- net /MCU_stm32_g431k8t6/NRST: track 10.9 -> 63.8 mm, vias 2 -> 4
- net /MCU_stm32_g431k8t6/FDCAN1_LED: track 9.13 -> 45.7 mm
- net /MCU_stm32_g431k8t6/JTDO_SWO: track 0.00 -> 36.1 mm
- net +24V: track 20.8 -> 56.3 mm
- net /MCU_stm32_g431k8t6/MCU_State_LED: track 10.1 -> 45.1 mm
- net /SPI_DAC/VOUT: track 5.83 -> 37.3 mm
- net /MCU_stm32_g431k8t6/JTCK_SWCLK: track 14.6 -> 36.7 mm
- net /MCU_stm32_g431k8t6/JTMS_SWDIO: track 16.4 -> 37.9 mm, vias 2 -> 3
- net /MCU_stm32_g431k8t6/ID_SW_BIT1: track 0.00 -> 18.7 mm, vias 1 -> 2
- net /MCU_stm32_g431k8t6/ID_SW_BIT2: track 2.61 -> 19.7 mm, vias 1 -> 2
- net /SPI_ADC/MOSI: track 0.00 -> 15.7 mm, vias 0 -> 1
- net /SPI_ADC/SCLK: track 0.00 -> 13.1 mm, vias 0 -> 1
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Other:
- board text added: "5V"
- board text added: "5VP"
- board text added: "CAN"
- board text added: "MCU"

Commit message: working
Parts:
- removed R28, R29, R39, R40, R43, R45: 0, Resistor_SMD:R_0603_1608Metric_Pad0.98x0.95mm_HandSolder
- added JP1: SolderJumper_2_Bridged, Jumper:SolderJumper-2_P1.3mm_Bridged2Bar_RoundedPad1.0x1.5mm, F.Cu at (163.8, 94.2)
- added JP2: SolderJumper_2_Bridged, Jumper:SolderJumper-2_P1.3mm_Bridged2Bar_RoundedPad1.0x1.5mm, F.Cu at (168.1, 92.8)
- added JP3: SolderJumper_3_Open, Jumper:SolderJumper-3_P1.3mm_Open_RoundedPad1.0x1.5mm_NumberLabels, F.Cu at (119.0, 95.2)
- added JP4: SolderJumper_3_Open, Jumper:SolderJumper-3_P1.3mm_Open_RoundedPad1.0x1.5mm_NumberLabels, F.Cu at (119.0, 98.5)
- added REF**: Y-robo_logo, y-robo_footprint:Y-robo_logo, F.Cu at (139.2, 79.5)
- moved R41 3.48 mm to (125.0, 98.5)
- moved R42 3.25 mm to (125.0, 95.5)
- turned R53 to 180 degrees
Connections:
- SW2 pad 3: unconnected-(SW2-Pad3) -> /MCU_stm32_g431k8t6/ID_SW_BIT3
- U1 pad 20: unconnected-(U1-PA10-Pad20) -> /MCU_stm32_g431k8t6/ID_SW_BIT3
Routing:
- net GNDPWR: track 3.64 -> 44.4 mm, vias 2 -> 136
- net +5VP: track 68.3 -> 92.1 mm
- net GND: track 17.4 -> 36.1 mm, vias 24 -> 122
- net /MCU_stm32_g431k8t6/ID_SW_BIT3: track 0.00 -> 17.0 mm, vias 0 -> 2
- net /SPI_Iso/CS2_IN: track 5.44 -> 12.9 mm
- net Net-(JP3-C): track 2.68 -> 8.02 mm
- net Net-(JP4-C): track 2.68 -> 7.77 mm
- net /Solenoid_Iso/PhotoRelay2_Drain: track 4.13 -> 7.62 mm
- net /SPI_DAC/OP_VIN+: track 13.3 -> 10.0 mm
- net /SPI_DAC/OP_VIN-: track 9.85 -> 6.60 mm
- net /SPI_DAC/VOUT: track 37.3 -> 40.5 mm
- net /SPI_Iso/CS1_IN: track 5.41 -> 8.61 mm
- net +12V: track 253.2 -> 250.1 mm
- net /MCU_stm32_g431k8t6/EP_Regu_ADC_CS: track 13.1 -> 10.5 mm
- net /MCU_stm32_g431k8t6/ID_SW_BIT2: track 19.7 -> 18.0 mm
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Other:
- outline, holes or cut-outs redrawn
- board text added: "+"
- board text added: "+VS"
- board text added: "-"
- board text added: "-VS"
- board text added: "0"
- board text added: "12V"
- board text added: "2026 YNCT Y-robo"
- board text added: "<-SENSE|LOCAL->"
- board text added: "CMD"
- board text added: "GND"
- board text added: "H"
- board text added: "L"
- board text added: "MON"
- board text added: "SD-Ver3.1"
- board text removed: "<-SENSE|LOCAL-> value: 0Ω"
